Commit message: chage the laser data plugin from gazebo_ros_laser to gazebo_ros_velodyne_laser

File: src/robot_description/urdf/t_robot.gazebo.xacro (robot description, xacro)
@@ -45,41 +45,44 @@
   </gazebo>
   <!-- robot laser setup in gazebo -->
-  <gazebo reference="robot_scan_link">
+  <gazebo reference="robot_laser_link">
     <material>Gazebo/Red</material>
-    <sensor type="ray" name="lds_lfcd_sensor">
-      <pose>0 0 0 0 0 0</pose>
-      <visualize>$(arg laser_visual)</visualize>
-      <update_rate>10</update_rate>
-      <ray>
-        <scan>
-          <vertical>
-            <samples>90</samples>
-            <resolution>1</resolution>
-            <min_angle>-0.2</min_angle>
-            <max_angle>+1.3</max_angle>
-          </vertical>
-          <!-- <horizontal>
-            <samples>90</samples>
-            <resolution>1</resolution>
-            <min_angle>-1.57</min_angle>
-            <max_angle>+1.57</max_angle>
-          </horizontal> -->
-        </scan>
-        <range>
-          <min>0.120</min>
-          <max>3.5</max>
-          <resolution>0.015</resolution>
-        </range>
-        <noise>
-          <type>gaussian</type>
-          <mean>0.0</mean>
-          <stddev>0.01</stddev>
-        </noise>
-      </ray>
-      <plugin name="gazebo_ros_lds_lfcd_controller" filename="libgazebo_ros_laser.so">
-        <topicName>scan</topicName>
-        <frameName>robot_scan_link</frameName>
-      </plugin>
-    </sensor>
+    <sensor type="ray" name="laser_16">
+        <pose>0 0 0 0 0 0</pose>
+        <visualize>true</visualize>
+        <update_rate>10</update_rate>
+        <ray>
+          <scan>
+            <horizontal>
+              <samples>90</samples>
+              <resolution>1</resolution>
+              <min_angle>-0.5</min_angle>
+              <max_angle>+0.5</max_angle>
+            </horizontal>
+            <vertical>
+              <samples>16</samples>
+              <resolution>1</resolution>
+              <min_angle>-${15.0*3.1415/180.0}</min_angle>
+              <max_angle> ${15.0*3.1415/180.0}</max_angle>
+            </vertical>
+          </scan>
+          <range>
+            <min>0.2</min>
+            <max>1</max>
+            <resolution>0.01</resolution>
+          </range>
+          <noise>
+            <type>gaussian</type>
+            <mean>0.0</mean>
+            <stddev>0.0</stddev>
+          </noise>
+        </ray>
+        <plugin name="gazebo_ros_laser_controller" filename="libgazebo_ros_velodyne_laser.so">
+          <topicName>/pointcloud222</topicName>
+          <frameName>robot_laser_link</frameName>
+          <min_range>0.2</min_range>
+          <max_range>1.0</max_range>
+          <gaussianNoise>0.008</gaussianNoise>
+        </plugin>
+      </sensor>
   </gazebo>
   <!-- 2 wheels -->

File: src/robot_description/urdf/t_robot.urdf.xacro (robot description, xacro)
@@ -42,11 +42,4 @@
     </inertial>
   </link>
-  <!-- joint of robot body link and laser -->
-  <joint name="body_scan_joint" type="continuous">
-    <parent link="robot_body_link"/>
-    <child link="robot_scan_link"/>
-    <origin xyz="0 0 ${height/2+0.01+lidar_above}" rpy="0 0 0"/>
-    <axis xyz="0 0 1"/>
-  </joint>
   <!-- imu joint -->
   <joint name="imu_joint" type="fixed">
@@ -57,6 +50,13 @@
   <!-- imu link -->
   <link name="imu_link"/>
+  <!-- joint of robot body link and laser -->
+  <joint name="body_scan_joint" type="fixed">
+    <parent link="robot_body_link"/>
+    <child link="robot_laser_link"/>
+    <origin xyz="0 0 ${height/2+0.01+lidar_above}" rpy="0 0 0"/>
+    <axis xyz="0 0 1"/>
+  </joint>
   <!-- laser sensor link -->
-  <link name="robot_scan_link">
+  <link name="robot_laser_link">
     <visual>
       <origin xyz="0.0 0.0 0.0" rpy="0 0 0"/>
@@ -80,5 +80,4 @@
     </inertial>
   </link>
-  <!-- TODO: the direction of the 2 wheels -->
   <!-- joint of robot body link and left wheel -->
   <joint name="wheel_left_joint" type="continuous">

Commit message: add ultrasound sensor

File: src/robot_description/urdf/t_robot.gazebo.xacro (robot description, xacro)
@@ -63,10 +63,10 @@
               <resolution>1</resolution>
               <min_angle>-${15.0*3.1415/180.0}</min_angle>
-              <max_angle> ${15.0*3.1415/180.0}</max_angle>
+              <max_angle>+${15.0*3.1415/180.0}</max_angle>
             </vertical>
           </scan>
           <range>
             <min>0.2</min>
-            <max>1</max>
+            <max>5</max>
             <resolution>0.01</resolution>
           </range>
@@ -81,5 +81,5 @@
           <frameName>robot_laser_link</frameName>
           <min_range>0.2</min_range>
-          <max_range>1.0</max_range>
+          <max_range>5.0</max_range>
           <gaussianNoise>0.008</gaussianNoise>
         </plugin>
@@ -144,8 +144,89 @@
       <wheelSeparation>0.46</wheelSeparation>
       <wheelDiameter>0.1</wheelDiameter>
-      <wheelAcceleration>1</wheelAcceleration>
+      <wheelAcceleration>100</wheelAcceleration>
       <wheelTorque>10</wheelTorque>
       <rosDebugLevel>na</rosDebugLevel>
     </plugin>
   </gazebo>
+  <!-- sonar plugin -->
+  <gazebo reference="sonar_01_link">
+    <material>Gazebo/ZincYellow</material>
+    <sensor type="ray" name="sonar_01_link">
+      <pose>0 0 0 0 0 0</pose>
+      <visualize>true</visualize>
+      <update_rate>5</update_rate>
+      <ray>
+        <scan>
+          <horizontal>
+            <samples>5</samples>
+            <resolution>1.0</resolution>
+            <min_angle>-0.25</min_angle>
+            <max_angle>0.25</max_angle>
+          </horizontal>
+          <vertical>
+            <samples>5</samples>
+            <resolution>1</resolution>
+            <min_angle>-0.25</min_angle>
+            <max_angle>0.25</max_angle>
+          </vertical>
+        </scan>
+        <range>
+          <min>0.03</min>
+          <max>0.2</max>
+          <resolution>0.01</resolution>
+        </range>
+      </ray>
+      <plugin name="sonar_01_plugin" filename="libgazebo_ros_range.so">
+        <gaussianNoise>0.005</gaussianNoise>
+        <alwaysOn>true</alwaysOn>
+        <updateRate>5</updateRate>
+        <topicName>sonar_01</topicName>
+        <frameName>sonar_01_link</frameName>
+        <!-- field of view = (max_angle - min_angle) -->
+        <!--               = 2 max_angle -->
+        <fov>0.5</fov>
+        <radiation>ultrasound</radiation>
+      </plugin>
+    </sensor>
+  </gazebo>
+  <gazebo reference="sonar_02_link">
+    <material>Gazebo/ZincYellow</material>
+    <sensor type="ray" name="sonar_02_link">
+      <pose>0 0 0 0 0 0</pose>
+      <visualize>true</visualize>
+      <update_rate>5</update_rate>
+      <ray>
+        <scan>
+          <horizontal>
+            <samples>5</samples>
+            <resolution>1.0</resolution>
+            <min_angle>-0.25</min_angle>
+            <max_angle>0.25</max_angle>
+          </horizontal>
+          <vertical>
+            <samples>5</samples>
+            <resolution>1</resolution>
+            <min_angle>-0.25</min_angle>
+            <max_angle>0.25</max_angle>
+          </vertical>
+        </scan>
+        <range>
+          <min>0.03</min>
+          <max>0.2</max>
+          <resolution>0.01</resolution>
+        </range>
+      </ray>
+      <plugin name="sonar_02_plugin" filename="libgazebo_ros_range.so">
+        <gaussianNoise>0.005</gaussianNoise>
+        <alwaysOn>true</alwaysOn>
+        <updateRate>5</updateRate>
+        <topicName>sonar_02</topicName>
+        <frameName>sonar_02_link</frameName>
+        <!-- field of view = (max_angle - min_angle) -->
+        <!--               = 2 max_angle -->
+        <fov>0.5</fov>
+        <radiation>ultrasound</radiation>
+      </plugin>
+    </sensor>
+  </gazebo>
 </robot>

File: src/robot_description/urdf/t_robot.urdf.xacro (robot description, xacro)
@@ -138,5 +138,5 @@
     </inertial>
   </link>
-  <!-- 2 caster wheel of front and back -->
+  <!-- caster back joint -->
   <joint name="caster_back_joint" type="fixed">
     <parent link="robot_body_link"/>
@@ -144,4 +144,5 @@
     <origin xyz="${-length/2} 0 ${-height/2-0.025}" rpy="0 0 0"/>
   </joint>
+  <!-- caseter back link -->
   <link name="caster_back_link">
     <visual>
@@ -172,4 +173,5 @@
     <origin xyz="${length/2} 0 ${-height/2-0.025}" rpy="0 0 0"/>
   </joint>
+  <!-- caster front link -->
   <link name="caster_front_link">
     <visual>
@@ -194,3 +196,61 @@
     </inertial>
   </link>
+  <!-- sonar joint -->
+  <joint name="sonar_01_joint" type="fixed">
+    <parent link="robot_body_link"/>
+    <child link="sonar_01_link"/>
+    <origin xyz="${length/6} ${width/2+0.01} 0" rpy="0 0 ${PI/2}"/>
+  </joint>
+  <!-- sonar link -->
+  <link name="sonar_01_link">
+    <visual>
+      <origin xyz="0 0 0" rpy="0 0 0"/>
+      <geometry>
+        <box size="0.01 0.01 0.01"/>
+      </geometry>
+      <material name="brown" />
+    </visual>
+    <collision>
+      <origin xyz="0 0 0" rpy="0 0 0"/>
+      <geometry>
+        <box size="0.01 0.01 0.01"/>
+      </geometry>
+    </collision>
+    <inertial>
+      <origin xyz="0 0 0" />
+      <mass value="0.001" />
+      <inertia ixx="0.001" ixy="0.0" ixz="0.0"
+               iyy="0.001" iyz="0.0"
+               izz="0.001" />
+    </inertial>
+  </link>
+  <!-- sonar joint -->
+  <joint name="sonar_02_joint" type="fixed">
+    <parent link="robot_body_link"/>
+    <child link="sonar_02_link"/>
+    <origin xyz="${length/6} ${-width/2-0.01} 0" rpy="0 0 ${-PI/2}"/>
+  </joint>
+  <!-- sonar link -->
+  <link name="sonar_02_link">
+    <visual>
+      <origin xyz="0 0 0" rpy="0 0 0"/>
+      <geometry>
+        <box size="0.01 0.01 0.01"/>
+      </geometry>
+      <material name="brown" />
+    </visual>
+    <collision>
+      <origin xyz="0 0 0" rpy="0 0 0"/>
+      <geometry>
+        <box size="0.01 0.01 0.01"/>
+      </geometry>
+    </collision>
+    <inertial>
+      <origin xyz="0 0 0" />
+      <mass value="0.001" />
+      <inertia ixx="0.001" ixy="0.0" ixz="0.0"
+               iyy="0.001" iyz="0.0"
+               izz="0.001" />
+    </inertial>
+  </link>
 </robot>

Commit message: add transmission part to xacro

File: src/robot_description/urdf/t_robot.gazebo.xacro (robot description, xacro)
@@ -56,12 +56,12 @@
               <samples>90</samples>
               <resolution>1</resolution>
-              <min_angle>-0.5</min_angle>
-              <max_angle>+0.5</max_angle>
+              <min_angle>-1.0</min_angle>
+              <max_angle>+1.0</max_angle>
             </horizontal>
             <vertical>
               <samples>16</samples>
               <resolution>1</resolution>
-              <min_angle>-${15.0*3.1415/180.0}</min_angle>
-              <max_angle>+${15.0*3.1415/180.0}</max_angle>
+              <min_angle>-${20.0*3.1415/180.0}</min_angle>
+              <max_angle>+${05.0*3.1415/180.0}</max_angle>
             </vertical>
           </scan>

File: src/robot_description/urdf/t_robot.urdf.xacro (robot description, xacro)
@@ -36,8 +36,8 @@
     <inertial>
       <origin xyz="0 0 0" rpy="0 0 0"/>
-      <mass value="8.2573504e-01"/>
-      <inertia ixx="2.2124416e-03" ixy="-1.2294101e-05" ixz="3.4938785e-05"
-               iyy="2.1193702e-03" iyz="-5.0120904e-06"
-               izz="2.0064271e-03" />
+      <mass value="100"/>
+      <inertia ixx="0.00001" ixy="0.00000" ixz="0.00000"
+               iyy="0.00001" iyz="0.00000"
+               izz="0.00001" />
     </inertial>
   </link>
@@ -73,5 +73,5 @@
     </collision>
     <inertial>
-      <mass value="0.114" />
+      <mass value="0.01" />
       <origin xyz="0 0 0" />
       <inertia ixx="0.001" ixy="0.0" ixz="0.0"
@@ -91,5 +91,5 @@
       <origin xyz="0.0 0.0 0.0" rpy="0 0 0"/>
       <geometry>
-        <cylinder length="0.02" radius="0.05"/>
+        <cylinder length="0.02" radius="0.1"/>
       </geometry>
       <material name="green"/>
@@ -98,15 +98,25 @@
       <origin xyz="0.0 0.0 0.0" rpy="0 0 0"/>
       <geometry>
-        <cylinder length="0.02" radius="0.05"/>
-      </geometry>
-    </collision>
-    <inertial>
-      <origin xyz="0 0 0" />
-      <mass value="2.8498940e-02" />
-      <inertia ixx="1.1175580e-05" ixy="-4.2369783e-11" ixz="-5.9381719e-09"
-               iyy="1.1192413e-05" iyz="-1.4400107e-11"
-               izz="2.0712558e-05" />
-    </inertial>
-  </link>
+        <cylinder length="0.02" radius="0.1"/>
+      </geometry>
+    </collision>
+    <inertial>
+      <origin xyz="0 0 0" />
+      <mass value="1" />
+      <inertia ixx="0.0025" ixy="0" ixz="0"
+               iyy="0.0025" iyz="0"
+               izz="0.005" />
+    </inertial>
+  </link>
+  <transmission name="wheel_left_trans">
+    <type>transmission_interface/SimpleTransmission</type>
+    <joint name="wheel_left_joint">
+      <hardwareInterface>VelocityJointInterface</hardwareInterface>
+    </joint>
+    <actuator name="wheel_left_motor">
+      <hardwareInterface>VelocityJointInterface</hardwareInterface>
+      <mechanicalReduction>1</mechanicalReduction>
+    </actuator>
+  </transmission>
   <!-- joint of robot body link and right wheel -->
   <joint name="wheel_right_joint" type="continuous">
@@ -120,5 +130,5 @@
       <origin xyz="0.0 0.0 0.0" rpy="0 0 0"/>
       <geometry>
-        <cylinder length="0.02" radius="0.05"/>
+        <cylinder length="0.02" radius="0.1"/>
       </geometry>
       <material name="green"/>
@@ -127,15 +137,25 @@
       <origin xyz="0.0 0.0 0.0" rpy="0 0 0"/>
       <geometry>
-        <cylinder length="0.02" radius="0.05"/>
-      </geometry>
-    </collision>
-    <inertial>
-      <origin xyz="0 0 0" />
-      <mass value="2.8498940e-02" />
-      <inertia ixx="1.1175580e-05" ixy="-4.2369783e-11" ixz="-5.9381719e-09"
-               iyy="1.1192413e-05" iyz="-1.4400107e-11"
-               izz="2.0712558e-05" />
-    </inertial>
-  </link>
+        <cylinder length="0.02" radius="0.1"/>
+      </geometry>
+    </collision>
+    <inertial>
+      <origin xyz="0 0 0" />
+      <mass value="1" />
+      <inertia ixx="0.0025" ixy="0" ixz="0"
+               iyy="0.0025" iyz="0"
+               izz="0.005" />
+    </inertial>
+  </link>
+  <transmission name="wheel_right_trans">
+    <type>transmission_interface/SimpleTransmission</type>
+    <joint name="wheel_right_joint">
+      <hardwareInterface>VelocityJointInterface</hardwareInterface>
+    </joint>
+    <actuator name="wheel_right_motor">
+      <hardwareInterface>VelocityJointInterface</hardwareInterface>
+      <mechanicalReduction>1</mechanicalReduction>
+    </actuator>
+  </transmission>
   <!-- caster back joint -->
   <joint name="caster_back_joint" type="fixed">
@@ -149,5 +169,5 @@
       <origin xyz="0 0 0" rpy="0 0 0"/>
       <geometry>
-        <box size="0.030 0.03 0.05"/>
+        <box size="0.030 0.03 0.10"/>
       </geometry>
       <material name="white" />
@@ -156,5 +176,5 @@
       <origin xyz="0 0 0" rpy="0 0 0"/>
       <geometry>
-        <box size="0.03 0.03 0.05"/>
+        <box size="0.03 0.03 0.10"/>
       </geometry>
     </collision>
@@ -178,12 +198,13 @@
       <origin xyz="0 0 0" rpy="0 0 0"/>
       <geometry>
-        <box size="0.03 0.03 0.05"/>
+        <box size="0.03 0.03 0.10"/>
       </geometry>
       <material name="white" />
     </visual>
-    <collision>
-      <origin xyz="0 0 0" rpy="0 0 0"/>
-      <geometry>
-        <box size="0.030 0.03 0.05"/>
+    c
+    <collision>
+      <origin xyz="0 0 0" rpy="0 0 0"/>
+      <geometry>
+        <box size="0.03 0.03 0.10"/>
       </geometry>
     </collision>

File: src/robot_description/urdf/t_robot_args.xacro (robot description, xacro)
@@ -27,5 +27,5 @@
   <!-- Distance between groud and robot which indicates the wheel's origin -->
   <!-- origin.z = wheel_radius - dis_robot_ground -->
-  <xacro:property name="dis_robot_groud" value="0.05"/>
+  <xacro:property name="dis_robot_groud" value="0.1"/>
   <!-- Distance between wheels and robot body side -->
   <!-- This arg determines the y coordinates of wheel -->

Commit message: update

File: src/robot_description/urdf/t_robot.gazebo.xacro (robot description, xacro)
@@ -109,6 +109,6 @@
   <!-- two caster wheels -->
   <gazebo reference="caster_back_link">
-    <mu1>0.0</mu1>
-    <mu2>0.0</mu2>
+    <mu1>0.000</mu1>
+    <mu2>0.000</mu2>
     <kp>1000000.0</kp>
     <kd>100.0</kd>
@@ -118,6 +118,6 @@
   </gazebo>
   <gazebo reference="caster_front_link">
-    <mu1>0.0</mu1>
-    <mu2>0.0</mu2>
+    <mu1>0.000</mu1>
+    <mu2>0.000</mu2>
     <kp>1000000.0</kp>
     <kd>100.0</kd>
@@ -143,5 +143,5 @@
       <rightJoint>wheel_right_joint</rightJoint>
       <wheelSeparation>0.46</wheelSeparation>
-      <wheelDiameter>0.1</wheelDiameter>
+      <wheelDiameter>0.2</wheelDiameter>
       <wheelAcceleration>100</wheelAcceleration>
       <wheelTorque>10</wheelTorque>

File: src/robot_description/urdf/t_robot.urdf.xacro (robot description, xacro)
@@ -17,5 +17,5 @@
     <parent link="base_world"/>
     <child link="robot_body_link"/>
-    <origin xyz="0.0 0.0 ${height/2 + dis_robot_groud - 0.01}" rpy="0 0 0"/>
+    <origin xyz="0.0 0.0 ${height/2 + wheel_radius - 0.01}" rpy="0 0 0"/>
   </joint>
   <!-- the robot body link -->
@@ -162,5 +162,5 @@
     <parent link="robot_body_link"/>
     <child link="caster_back_link"/>
-    <origin xyz="${-length/2} 0 ${-height/2-0.025}" rpy="0 0 0"/>
+    <origin xyz="${-length/2} 0 ${-height/2-0.05}" rpy="0 0 0"/>
   </joint>
   <!-- caseter back link -->
@@ -181,5 +181,5 @@
     <inertial>
       <origin xyz="0 0 0" />
-      <mass value="0.005" />
+      <mass value="1" />
       <inertia ixx="0.001" ixy="0.0" ixz="0.0"
                iyy="0.001" iyz="0.0"
@@ -191,5 +191,5 @@
     <parent link="robot_body_link"/>
     <child link="caster_front_link"/>
-    <origin xyz="${length/2} 0 ${-height/2-0.025}" rpy="0 0 0"/>
+    <origin xyz="${length/2} 0 ${-height/2-0.05}" rpy="0 0 0"/>
   </joint>
   <!-- caster front link -->
@@ -202,5 +202,4 @@
       <material name="white" />
     </visual>
-    c
     <collision>
       <origin xyz="0 0 0" rpy="0 0 0"/>
@@ -211,5 +210,5 @@
     <inertial>
       <origin xyz="0 0 0" />
-      <mass value="0.005" />
+      <mass value="1" />
       <inertia ixx="0.001" ixy="0.0" ixz="0.0"
                iyy="0.001" iyz="0.0"

File: src/robot_description/urdf/t_robot_args.xacro (robot description, xacro)
@@ -8,5 +8,5 @@
   <!-- *********************************** -->
   <xacro:property name="PI" value="3.1415926535897931"/>
-  <xacro:property name="mass" value="1"/>
+  <xacro:property name="mass" value="20"/>
   <!-- Robot body is a box, below is width, height, length of the box -->
   <!-- Length by x axis, width by y axis, height by z axis -->
@@ -25,7 +25,4 @@
   <xacro:property name="caster_thickness" value="0.01"/>
   <xacro:property name="caster_radius" value="0.01"/>
-  <!-- Distance between groud and robot which indicates the wheel's origin -->
-  <!-- origin.z = wheel_radius - dis_robot_ground -->
-  <xacro:property name="dis_robot_groud" value="0.1"/>
   <!-- Distance between wheels and robot body side -->
   <!-- This arg determines the y coordinates of wheel -->
