Commit message: macro-mid

File: src/robot_description/urdf/parts/caster_model.xacro (robot description, xacro)
@@ -2,5 +2,5 @@
 <robot xmlns:xacro="TergeoRobot" name="tergeo">
   <!-- args -->
-  <xacro:property name="caster_height" value=" 0.1" />
+  <xacro:property name="caster_height" value=" 0.05" />
   <xacro:property name="caster_length" value="0.03" />
   <xacro:property name="caster_width" value="0.03" />
@@ -37,6 +37,6 @@
     <!-- gazebo element -->
     <gazebo reference="${caster_name}_link">
-      <mu1>0.000</mu1>
-      <mu2>0.000</mu2>
+      <mu1>0.001</mu1>
+      <mu2>0.001</mu2>
       <kp>1000000.0</kp>
       <kd>100.0</kd>

File: src/robot_description/urdf/parts/lidar_model.xacro (robot description, xacro)
@@ -5,15 +5,15 @@
   <xacro:property name="lidar_height" value="0.02" />
   <xacro:property name="lidar_radius" value="0.02" />
-  <xacro:property name="h_sample" value="90" />
-  <xacro:property name="h_min_angle" value="-1.0" />
-  <xacro:property name="h_max_angle" value="1.0" />
+  <xacro:property name="h_sample" value="1800" />
+  <xacro:property name="h_min_angle" value="${-180*3.1415/180.0}" />
+  <xacro:property name="h_max_angle" value="${+180*3.1415/180.0}" />
   <xacro:property name="v_sample" value="16" />
-  <xacro:property name="v_min_angle" value="${-5.0*3.1415/180.0}" />
-  <xacro:property name="v_max_angle" value="${30*3.1415/180.0}" />
-  <xacro:property name="pub_topic_name" value="/pointcloud_gazebo" />
+  <xacro:property name="v_min_angle" value="${-15.0*3.1415/180.0}" />
+  <xacro:property name="v_max_angle" value="${15*3.1415/180.0}" />
+  <xacro:property name="pub_topic_name" value="/sensor/lidar16/top/pointcloud" />
   <xacro:property name="min_range" value="0.2" />
-  <xacro:property name="max_range" value="5.0" />
+  <xacro:property name="max_range" value="10.0" />
   <xacro:property name="min_intensity" value="0.001" />
-  <xacro:property name="gaussian_noise" value="0.08" />
+  <xacro:property name="gaussian_noise" value="0.02" />
   <!-- Macro to generate lidar -->
   <xacro:macro name="lidar_model" params="lidar_name parent_link lidar_xyz lidar_rpy lidar_axis">
@@ -52,5 +52,5 @@
       <sensor type="ray" name="laser_16">
         <pose>0 0 0 0 0 0</pose>
-        <visualize>true</visualize>
+        <visualize>false</visualize>
         <update_rate>10</update_rate>
         <ray>

File: src/robot_description/urdf/parts/wheel_model.xacro (robot description, xacro)
@@ -3,5 +3,5 @@
   <!-- args -->
   <xacro:property name="wheel_thickness" value=" 0.02" />
-  <xacro:property name="wheel_radius" value="0.1" />
+  <xacro:property name="wheel_radius" value="0.05" />
   <!-- Definition of the wheel macro -->
   <xacro:macro name="wheel_model" params="wheel_name parent_link wheel_xyz wheel_rpy wheel_axis">
@@ -28,5 +28,5 @@
         </geometry>
       </collision>
-      <!-- <inertial>
+      <inertial>
         <origin xyz="0 0 0" />
         <mass value="1" />
@@ -34,6 +34,6 @@
                 iyy="0.0025" iyz="0"
                 izz="0.005" />
-      </inertial> -->
-      <inertial>
+      </inertial>
+      <!-- <inertial>
         <origin xyz="0 0 0" />
         <mass value="2" />
@@ -41,5 +41,5 @@
                 iyy="${0.025/2}" iyz="0"
                 izz="${0.05/2}" />
-      </inertial>
+      </inertial> -->
     </link>
     <!-- setup the motor -->
@@ -87,5 +87,5 @@
         <wheelDiameter>${2*wheel_radius}</wheelDiameter>
         <wheelAcceleration>100</wheelAcceleration>
-        <wheelTorque>10</wheelTorque>
+        <wheelTorque>5</wheelTorque>
         <rosDebugLevel>na</rosDebugLevel>
       </plugin>

File: src/robot_description/urdf/t_robot_args.xacro (robot description, xacro)
@@ -23,5 +23,5 @@
   <!-- Assign the attribute for thickness and radius -->
   <xacro:property name="wheel_thickness" value="0.02"/>
-  <xacro:property name="wheel_radius" value="0.1"/>
+  <xacro:property name="wheel_radius" value="0.05"/>
   <xacro:property name="caster_thickness" value="0.01"/>
   <xacro:property name="caster_radius" value="0.01"/>

File: src/robot_description/urdf/tergeo.urdf.xacro (robot description, xacro)
@@ -9,7 +9,7 @@
   <xacro:include filename="$(find robot_description)/urdf/parts/*.xacro"/>
   <!-- This macro generates a ${body_name}_link -->
-  <xacro:base_world world_name="base_world" body_name="body" mass="${mass}" length="${length}" width="${width}" height="${height}" above_groud_height="${above_groud_height}"/>
+  <xacro:base_world world_name="base_world" body_name="body" mass="${mass}" length="${length}" width="${width}" height="${height}" above_groud_height="${above_groud_height}" />
   <!-- This macro generates the lidar model -->
-  <xacro:lidar_model lidar_name="top_lidar16" parent_link="body_link" lidar_xyz="0 0 ${lidar_above+height/2}" lidar_rpy="0 0 0" lidar_axis="0 0 1"/>
+  <xacro:lidar_model lidar_name="top_lidar16" parent_link="body_link" lidar_xyz="0 0 ${lidar_above+height/2}" lidar_rpy="0 0 0" lidar_axis="0 0 1" />
   <!-- This macro generates left wheel -->
   <xacro:wheel_model wheel_name="left_wheel" parent_link="body_link" wheel_xyz="0.0 ${width/2+0.02} ${-height/2}" wheel_rpy="${-PI/2} 0 0" wheel_axis="0 0 1" />
@@ -19,11 +19,11 @@
   <xacro:wheel_control left_wheel_name="left_wheel" right_wheel_name="right_wheel" />
   <!-- This macro generates front caster -->
-  <xacro:caster_model caster_name="front_caster" parent_link="body_link" caster_xyz="${length/2} 0 ${-height/2-0.05}" caster_rpy="0 0 0" />
+  <xacro:caster_model caster_name="front_caster" parent_link="body_link" caster_xyz="${length/2} 0 ${-height/2-0.025}" caster_rpy="0 0 0" />
   <!-- This macro generates back caster -->
-  <xacro:caster_model caster_name="back_caster" parent_link="body_link" caster_xyz="${-length/2} 0 ${-height/2-0.05}" caster_rpy="0 0 0" />
+  <xacro:caster_model caster_name="back_caster" parent_link="body_link" caster_xyz="${-length/2} 0 ${-height/2-0.025}" caster_rpy="0 0 0" />
   <!-- This macro generates left sonar -->
-  <xacro:sonar_model sonar_name="left_sonar" parent_link="body_link" sonar_xyz="0 ${width/2+0.01} 0" sonar_rpy="0 0 ${PI/2}" />
+  <!-- <xacro:sonar_model sonar_name="left_sonar" parent_link="body_link" sonar_xyz="0 ${width/2+0.01} 0" sonar_rpy="0 0 ${PI/2}" /> -->
   <!-- This macro generates right sonar -->
-  <xacro:sonar_model sonar_name="right_sonar" parent_link="body_link" sonar_xyz="0 ${-width/2-0.01} 0" sonar_rpy="0 0 ${-PI/2}" />
+  <!-- <xacro:sonar_model sonar_name="right_sonar" parent_link="body_link" sonar_xyz="0 ${-width/2-0.01} 0" sonar_rpy="0 0 ${-PI/2}" /> -->
   <!-- This macro generates imu -->
   <xacro:imu_model imu_name="imu" parent_link="body_link" imu_xyz="0 0 0" imu_rpy="0 0 0" />

Commit message: update

File: src/robot_description/urdf/parts/caster_model.xacro (robot description, xacro)
@@ -2,5 +2,5 @@
 <robot xmlns:xacro="TergeoRobot" name="tergeo">
   <!-- args -->
-  <xacro:property name="caster_height" value=" 0.05" />
+  <xacro:property name="caster_height" value=" 0.10" />
   <xacro:property name="caster_length" value="0.03" />
   <xacro:property name="caster_width" value="0.03" />

File: src/robot_description/urdf/parts/lidar_model.xacro (robot description, xacro)
@@ -6,12 +6,12 @@
   <xacro:property name="lidar_radius" value="0.02" />
   <xacro:property name="h_sample" value="1800" />
-  <xacro:property name="h_min_angle" value="${-180*3.1415/180.0}" />
-  <xacro:property name="h_max_angle" value="${+180*3.1415/180.0}" />
+  <xacro:property name="h_min_angle" value="${-180*3.1415926535897931/180.0}" />
+  <xacro:property name="h_max_angle" value="${+180*3.1415926535897931/180.0}" />
   <xacro:property name="v_sample" value="16" />
-  <xacro:property name="v_min_angle" value="${-15.0*3.1415/180.0}" />
-  <xacro:property name="v_max_angle" value="${15*3.1415/180.0}" />
+  <xacro:property name="v_min_angle" value="${-15.0*3.1415926535897931/180.0}" />
+  <xacro:property name="v_max_angle" value="${15.0*3.1415926535897931/180.0}" />
   <xacro:property name="pub_topic_name" value="/sensor/lidar16/top/pointcloud" />
   <xacro:property name="min_range" value="0.2" />
-  <xacro:property name="max_range" value="10.0" />
+  <xacro:property name="max_range" value="100.0" />
   <xacro:property name="min_intensity" value="0.001" />
   <xacro:property name="gaussian_noise" value="0.02" />

File: src/robot_description/urdf/parts/wheel_model.xacro (robot description, xacro)
@@ -3,5 +3,5 @@
   <!-- args -->
   <xacro:property name="wheel_thickness" value=" 0.02" />
-  <xacro:property name="wheel_radius" value="0.05" />
+  <xacro:property name="wheel_radius" value="0.10" />
   <!-- Definition of the wheel macro -->
   <xacro:macro name="wheel_model" params="wheel_name parent_link wheel_xyz wheel_rpy wheel_axis">

File: src/robot_description/urdf/tergeo.urdf.xacro (robot description, xacro)
@@ -19,7 +19,7 @@
   <xacro:wheel_control left_wheel_name="left_wheel" right_wheel_name="right_wheel" />
   <!-- This macro generates front caster -->
-  <xacro:caster_model caster_name="front_caster" parent_link="body_link" caster_xyz="${length/2} 0 ${-height/2-0.025}" caster_rpy="0 0 0" />
+  <xacro:caster_model caster_name="front_caster" parent_link="body_link" caster_xyz="${length/2} 0 ${-height/2-0.05}" caster_rpy="0 0 0" />
   <!-- This macro generates back caster -->
-  <xacro:caster_model caster_name="back_caster" parent_link="body_link" caster_xyz="${-length/2} 0 ${-height/2-0.025}" caster_rpy="0 0 0" />
+  <xacro:caster_model caster_name="back_caster" parent_link="body_link" caster_xyz="${-length/2} 0 ${-height/2-0.05}" caster_rpy="0 0 0" />
   <!-- This macro generates left sonar -->
   <!-- <xacro:sonar_model sonar_name="left_sonar" parent_link="body_link" sonar_xyz="0 ${width/2+0.01} 0" sonar_rpy="0 0 ${PI/2}" /> -->

Commit message: finished base config include macro

File: src/robot_description/urdf/parts/caster_model.xacro (robot description, xacro)
@@ -1,14 +1,19 @@
 <?xml version="1.0"?>
 <robot xmlns:xacro="TergeoRobot" name="tergeo">
-  <!-- args -->
-  <xacro:property name="caster_height" value=" 0.10" />
-  <xacro:property name="caster_length" value="0.03" />
-  <xacro:property name="caster_width" value="0.03" />
-  <!-- TODO: need external args -->
-  <xacro:macro name="caster_model" params="caster_name parent_link caster_xyz caster_rpy">
+  <!-- Import args -->
+  <xacro:include filename="$(find robot_description)/urdf/parts_cfg/base_world_cfg.xacro" ns="base" />
+  <xacro:include filename="$(find robot_description)/urdf/parts_cfg/wheel_cfg.xacro" ns="wheel" />
+  <xacro:include filename="$(find robot_description)/urdf/parts_cfg/caster_cfg.xacro" ns="caster" />
+  <xacro:macro name="caster_model" params="caster_name parent_link">
+    <xacro:if value="${'back' in caster_name}">
+      <xacro:property name="caster_xyz" value="${-(base.length/2)} 0 ${-(base.height/2+caster.height/2-wheel.z_dis)}" />
+    </xacro:if>
+    <xacro:if value="${'front' in caster_name}">
+      <xacro:property name="caster_xyz" value="${+(base.length/2)} 0 ${-(base.height/2+caster.height/2-wheel.z_dis)}" />
+    </xacro:if>
     <joint name="${caster_name}_joint" type="fixed">
       <parent link="${parent_link}"/>
       <child link="${caster_name}_link"/>
-      <origin xyz="${caster_xyz}" rpy="${caster_rpy}"/>
+      <origin xyz="${caster_xyz}" rpy="${caster.rpy}"/>
     </joint>
     <!-- caseter link -->
@@ -17,5 +22,5 @@
         <origin xyz="0 0 0" rpy="0 0 0"/>
         <geometry>
-          <box size="${caster_length} ${caster_width} ${caster_height}"/>
+          <box size="${caster.length} ${caster.width} ${caster.height}"/>
         </geometry>
         <material name="white" />
@@ -24,10 +29,10 @@
         <origin xyz="0 0 0" rpy="0 0 0"/>
         <geometry>
-          <box size="${caster_length} ${caster_width} ${caster_height}"/>
+          <box size="${caster.length} ${caster.width} ${caster.height}"/>
         </geometry>
       </collision>
       <inertial>
         <origin xyz="0 0 0" />
-        <mass value="1" />
+        <mass value="${caster.mass}" />
         <inertia ixx="0.000" ixy="0.0" ixz="0.0"
                  iyy="0.000" iyz="0.0"
@@ -37,10 +42,10 @@
     <!-- gazebo element -->
     <gazebo reference="${caster_name}_link">
-      <mu1>0.001</mu1>
-      <mu2>0.001</mu2>
-      <kp>1000000.0</kp>
-      <kd>100.0</kd>
-      <minDepth>0.001</minDepth>
-      <maxVel>1.0</maxVel>
+      <mu1>${caster.mu1}</mu1>
+      <mu2>${caster.mu2}</mu2>
+      <kp>${caster.kp}</kp>
+      <kd>${caster.kd}</kd>
+      <minDepth>${caster.min_depth}</minDepth>
+      <maxVel>${caster.max_vel}</maxVel>
       <material>Gazebo/FlatBlack</material>
     </gazebo>

File: src/robot_description/urdf/parts/lidar_model.xacro (robot description, xacro)
@@ -3,8 +3,4 @@
   <!-- base cfg and lidar cfg -->
   <xacro:include filename="$(find robot_description)/urdf/parts_cfg/lidar_cfg.xacro" ns="lidar" />
-  <xacro:include filename="$(find robot_description)/urdf/parts_cfg/base_world_cfg.xacro" ns="base" />
-  <!-- local args which need args from base cfg and lidar cfg -->
-  <!-- This arg will be deprecated soon -->
-  <xacro:property name="lidar_xyz" value="0 0 ${lidar.above_height+base.height/2+lidar.height/2}" />
   <!-- Macro to generate lidar model -->
   <xacro:macro name="lidar_model" params="lidar_name parent_link">
@@ -12,5 +8,5 @@
       <parent link="${parent_link}" />
       <child link="${lidar_name}_link" />
-      <origin xyz="${lidar_xyz}" rpy="${lidar.rpy}" />
+      <origin xyz="${lidar.xyz}" rpy="${lidar.rpy}" />
       <axis xyz="${lidar.axis}" />
     </joint>

File: src/robot_description/urdf/parts/wheel_model.xacro (robot description, xacro)
@@ -2,16 +2,14 @@
 <robot xmlns:xacro="TergeoRobot" name="tergeo">
   <!-- include corresponding config file -->
+  <xacro:include filename="$(find robot_description)/urdf/parts_cfg/base_world_cfg.xacro" ns="base" />
   <xacro:include filename="$(find robot_description)/urdf/parts_cfg/wheel_cfg.xacro" ns="wheel" />
-  <xacro:include filename="$(find robot_description)/urdf/parts_cfg/base_world_cfg.xacro" ns="base" />
   <!-- Definition of the wheel macro -->
-  <xacro:macro name="wheel_model" params="wheel_name parent_link wheel_xyz wheel_rpy wheel_axis">
+  <xacro:macro name="wheel_model" params="wheel_name parent_link">
     <!-- args depend on macro params and cfg file -->
     <xacro:if value="${'left' in wheel_name}">
-      <xacro:property name="wheel_xyz" value="0 +" />
-      <xacro:property name="wheel_rpy" value="" />
+      <xacro:property name="wheel_xyz" value="0 ${+(base.width/2+wheel.thickness/2+wheel.y_dis)} ${-base.height/2+wheel.z_dis}" />
     </xacro:if>
     <xacro:if value="${'right' in wheel_name}">
-      <xacro:property name="wheel_xyz" value="" />
-      <xacro:property name="wheel_rpy" value="" />
+      <xacro:property name="wheel_xyz" value="0 ${-(base.width/2+wheel.thickness/2+wheel.y_dis)} ${-base.height/2+wheel.z_dis}" />
     </xacro:if>
     <!-- wheel joint -->
@@ -19,6 +17,6 @@
       <parent link="${parent_link}" />
       <child link="${wheel_name}_link" />
-      <origin xyz="${wheel_xyz}" rpy="${wheel_rpy}" />
-      <axis xyz="${wheel_axis}" />
+      <origin xyz="${wheel_xyz}" rpy="${wheel.rpy}" />
+      <axis xyz="${wheel.axis}" />
     </joint>
     <!-- wheel link -->
@@ -39,8 +37,8 @@
       <inertial>
         <origin xyz="0 0 0" />
-        <mass value="${}" />
-        <inertia ixx="0.0025" ixy="0" ixz="0"
-                iyy="0.0025" iyz="0"
-                izz="0.005" />
+        <mass value="${wheel.mass}" />
+        <inertia ixx="${wheel.ixxiyy}" ixy="0" ixz="0"
+                 iyy="${wheel.ixxiyy}" iyz="0"
+                 izz="${wheel.izz}" />
       </inertial>
     </link>
@@ -58,11 +56,11 @@
     <!-- gazebo element -->
     <gazebo reference="${wheel_name}_link">
-      <mu1>0.1</mu1>
-      <mu2>0.1</mu2>
-      <kp>500000.0</kp>
-      <kd>10.0</kd>
-      <minDepth>0.001</minDepth>
-      <maxVel>1.0</maxVel>
-      <fdir1>1 0 0</fdir1>
+      <mu1>${wheel.mu1}</mu1>
+      <mu2>${wheel.mu2}</mu2>
+      <kp>${wheel.kp}</kp>
+      <kd>${wheel.kd}</kd>
+      <minDepth>${wheel.min_depth}</minDepth>
+      <maxVel>${wheel.max_vel}</maxVel>
+      <fdir1>${wheel.fdir1}</fdir1>
       <material>Gazebo/Green</material>
     </gazebo>
@@ -72,8 +70,8 @@
     <gazebo>
       <plugin name="robot_controller" filename="libgazebo_ros_diff_drive.so">
-        <commandTopic>cmd_vel</commandTopic>
-        <odometryTopic>odom</odometryTopic>
-        <odometryFrame>odom</odometryFrame>
-        <odometrySource>world</odometrySource>
+        <commandTopic>${wheel.sub_cmd_topic}</commandTopic>
+        <odometryTopic>${wheel.pub_odom_topic}</odometryTopic>
+        <odometryFrame>${wheel.odom_frame}</odometryFrame>
+        <odometrySource>${wheel.odom_src}</odometrySource>
         <publishOdomTF>true</publishOdomTF>
         <robotBaseFrame>base_world</robotBaseFrame>
@@ -82,12 +80,11 @@
         <publishWheelJointState>true</publishWheelJointState>
         <legacyMode>false</legacyMode>
-        <updateRate>30</updateRate>
+        <updateRate>${wheel.update_rate}</updateRate>
         <leftJoint>${left_wheel_name}_joint</leftJoint>
         <rightJoint>${right_wheel_name}_joint</rightJoint>
-        <!-- wheel seperation need to know the body width -->
-        <wheelSeparation>0.46</wheelSeparation>
+        <wheelSeparation>${base.width+2*wheel.thickness/2+2*wheel.y_dis}</wheelSeparation>
         <wheelDiameter>${2*wheel.radius}</wheelDiameter>
-        <wheelAcceleration>100</wheelAcceleration>
-        <wheelTorque>5</wheelTorque>
+        <wheelAcceleration>${wheel.accel}</wheelAcceleration>
+        <wheelTorque>${wheel.torque}</wheelTorque>
         <rosDebugLevel>na</rosDebugLevel>
       </plugin>

File: src/robot_description/urdf/parts_cfg/base_world_cfg.xacro (robot description, xacro)
@@ -7,4 +7,4 @@
   <xacro:property name="width" value="0.4" />
   <xacro:property name="height" value="0.3" />
-  <xacro:property name="above_groud_height" value="0.2" />
+  <xacro:property name="above_groud_height" value="0.05" />
 </robot>

File: src/robot_description/urdf/parts_cfg/lidar_cfg.xacro (robot description, xacro)
@@ -1,4 +1,6 @@
 <?xml version="1.0"?>
 <robot name="tergeo" xmlns:xacro="TergeoRobot">
+  <!-- Import the cfg -->
+  <xacro:include filename="$(find robot_description)/urdf/parts_cfg/base_world_cfg.xacro" ns="base" />
   <!-- Math args -->
   <xacro:property name="PI" value="3.1415926535897931" />
@@ -7,10 +9,10 @@
   <xacro:property name="height" value="0.02" />
   <xacro:property name="radius" value="0.02" />
+  <!-- This arg will be deprecated soon -->
+  <xacro:property name="above_height" value="0.15" />
   <!-- TODO: xyz -->
-  <xacro:property name="xyz" value="0 0 0" />
+  <xacro:property name="xyz" value="0 0 ${above_height+base.height/2+height/2}" />
   <xacro:property name="rpy" value="0 0 0" />
   <xacro:property name="axis" value="0 0 1" />
-  <!-- This arg will be deprecated soon -->
-  <xacro:property name="above_height" value="0.15" />
   <!-- Lidar intrinsic -->
   <xacro:property name="h_sample" value="180" />

File: src/robot_description/urdf/parts_cfg/wheel_cfg.xacro (robot description, xacro)
@@ -1,13 +1,33 @@
 <?xml version="1.0"?>
 <robot name="tergeo" xmlns:xacro="TergeoRobot">
-  <xacro:property name="left_xyz" value="" />
-  <xacro:property name="left_rpy" value="" />
-  <xacro:property name="right_xyz" value="" />
-  <xacro:property name="right_rpy" value="" />
+  <!-- Math args -->
+  <xacro:property name="PI" value="3.1415926535897931" />
+  <!-- Wheel extrinsic -->
+  <xacro:property name="rpy" value="${-PI/2} 0 0" />
   <xacro:property name="axis" value="0 0 1" />
   <xacro:property name="mass" value="1.00" />
   <xacro:property name="thickness" value="0.02" />
   <xacro:property name="radius" value="0.10" />
-  <xacro:property name="ixx_iyy" value="${mass*(3*radius*radius+thickness*thickness)/12}" />
+  <!-- <xacro:property name="ixxiyy" value="0.0" />
+  <xacro:property name="izz" value="0.0" /> -->
+  <xacro:property name="ixxiyy" value="${mass*(3*radius*radius+thickness*thickness)/12}" />
   <xacro:property name="izz" value="${mass*radius*radius/2}" />
+  <xacro:property name="y_dis" value="0.01" />
+  <xacro:property name="z_dis" value="0.05" />
+  <!-- Wheel intrinsic -->
+  <xacro:property name="mu1" value="0.1" />
+  <xacro:property name="mu2" value="0.1" />
+  <xacro:property name="kp" value="500000.0" />
+  <xacro:property name="kd" value="10.0" />
+  <xacro:property name="min_depth" value="0.001" />
+  <xacro:property name="max_vel" value="10.0" />
+  <xacro:property name="fdir1" value="1 0 0" />
+  <!-- Control args -->
+  <xacro:property name="sub_cmd_topic" value="cmd_vel" />
+  <xacro:property name="pub_odom_topic" value="odom" />
+  <xacro:property name="odom_frame" value="odom" />
+  <xacro:property name="odom_src" value="world" />
+  <xacro:property name="update_rate" value="30" />
+  <xacro:property name="accel" value="1000" />
+  <xacro:property name="torque" value="5" />
 </robot>

File: src/robot_description/urdf/tergeo.urdf.xacro (robot description, xacro)
@@ -13,13 +13,13 @@
   <xacro:lidar_model lidar_name="top_lidar16" parent_link="body_link" />
   <!-- This macro generates left wheel -->
-  <!-- <xacro:wheel_model wheel_name="left_wheel" parent_link="body_link" wheel_xyz="0.0 ${width/2+0.02} ${-height/2}" wheel_rpy="${-PI/2} 0 0" wheel_axis="0 0 1" /> -->
+  <xacro:wheel_model wheel_name="left_wheel" parent_link="body_link" />
   <!-- This macro generates right wheel -->
-  <!-- <xacro:wheel_model wheel_name="right_wheel" parent_link="body_link" wheel_xyz="0.0 ${-width/2-0.02} ${-height/2}" wheel_rpy="${-PI/2} 0 0" wheel_axis="0 0 1" /> -->
+  <xacro:wheel_model wheel_name="right_wheel" parent_link="body_link" />
   <!-- This macro setups the control -->
-  <!-- <xacro:wheel_control left_wheel_name="left_wheel" right_wheel_name="right_wheel" /> -->
+  <xacro:wheel_control left_wheel_name="left_wheel" right_wheel_name="right_wheel" />
   <!-- This macro generates front caster -->
-  <!-- <xacro:caster_model caster_name="front_caster" parent_link="body_link" caster_xyz="${length/2} 0 ${-height/2-0.05}" caster_rpy="0 0 0" /> -->
+  <xacro:caster_model caster_name="front_caster" parent_link="body_link" />
   <!-- This macro generates back caster -->
-  <!-- <xacro:caster_model caster_name="back_caster" parent_link="body_link" caster_xyz="${-length/2} 0 ${-height/2-0.05}" caster_rpy="0 0 0" /> -->
+  <xacro:caster_model caster_name="back_caster" parent_link="body_link" />
   <!-- This macro generates left sonar -->
   <!-- <xacro:sonar_model sonar_name="left_sonar" parent_link="body_link" sonar_xyz="0 ${width/2+0.01} 0" sonar_rpy="0 0 ${PI/2}" /> -->
