Commit message: add imu_cfg and sonar_cfg

File: src/robot_description/urdf/parts/imu_model.xacro (robot description, xacro)
@@ -2,8 +2,7 @@
 <robot xmlns:xacro="TergeoRobot" name="tergeo">
   <!-- args -->
-  <xacro:property name="imu_topic_name" value="imu" />
-  <xacro:property name="imu_service_name" value="imu_service" />
+  <xacro:include filename="$(find robot_description)/urdf/parts_cfg/imu_cfg.xacro" ns="imu" />
   <!-- Macro definition -->
-  <xacro:macro name="imu_model" params="imu_name parent_link imu_xyz imu_rpy">
+  <xacro:macro name="imu_model" params="imu_name parent_link">
     <!-- imu joint -->
     <joint name="${imu_name}_joint" type="fixed">
@@ -25,25 +24,25 @@
     <gazebo>
       <plugin name="${imu_name}_plugin" filename="libgazebo_ros_imu.so">
-        <alwaysOn>true</alwaysOn>
+        <alwaysOn>${imu.always_on}</alwaysOn>
         <bodyName>${imu_name}_link</bodyName>
         <frameName>${imu_name}_link</frameName>
-        <topicName>${imu_topic_name}</topicName>
-        <serviceName>${imu_service_name}</serviceName>
-        <gaussianNoise>0.0</gaussianNoise>
-        <updateRate>60</updateRate>
+        <topicName>${imu.topic_name}</topicName>
+        <serviceName>${imu.service_name}</serviceName>
+        <gaussianNoise>${imu.g_noise}</gaussianNoise>
+        <updateRate>${imu.update_rate}</updateRate>
         <imu>
           <noise>
             <type>gaussian</type>
             <rate>
-              <mean>0.0</mean>
-              <stddev>2e-4</stddev>
-              <bias_mean>0.0000075</bias_mean>
-              <bias_stddev>0.0000008</bias_stddev>
+              <mean>${imu.rate_mean}</mean>
+              <stddev>${imu.rate_std}</stddev>
+              <bias_mean>${imu.rate_bias_mean}</bias_mean>
+              <bias_stddev>${imu.rate_bias_std}</bias_stddev>
             </rate>
             <accel>
-              <mean>0.0</mean>
-              <stddev>1.7e-2</stddev>
-              <bias_mean>0.1</bias_mean>
-              <bias_stddev>0.001</bias_stddev>
+              <mean>${imu.acc_mean}</mean>
+              <stddev>${imu.acc_std}</stddev>
+              <bias_mean>${imu.acc_bias_mean}</bias_mean>
+              <bias_stddev>${imu.acc_bias_std}</bias_stddev>
             </accel>
           </noise>

File: src/robot_description/urdf/parts/sonar_model.xacro (robot description, xacro)
@@ -1,5 +1,14 @@
 <?xml version="1.0"?>
 <robot xmlns:xacro="TergeoRobot" name="tergeo">
-<xacro:macro name="sonar_model" params="sonar_name parent_link sonar_xyz sonar_rpy">
+<xacro:include filename="$(find robot_description)/urdf/parts_cfg/sonar_cfg.xacro" ns="sonar" />
+<xacro:macro name="sonar_model" params="sonar_name parent_link">
+  <xacro:if value="${'left' in sonar_name}">
+      <xacro:property name="sonar_xyz" value="${sonar.left_xyz}" />
+      <xacro:property name="sonar_rpy" value="${sonar.left_rpy}" />
+  </xacro:if>
+  <xacro:if value="${'right' in sonar_name}">
+      <xacro:property name="sonar_xyz" value="${sonar.right_xyz}" />
+      <xacro:property name="sonar_rpy" value="${sonar.right_rpy}" />
+  </xacro:if>
   <!-- sonar joint -->
   <joint name="${sonar_name}_joint" type="fixed">
@@ -37,36 +46,34 @@
     <sensor type="ray" name="${sonar_name}">
       <pose>0 0 0 0 0 0</pose>
-      <visualize>true</visualize>
-      <update_rate>5</update_rate>
+      <visualize>${sonar.visualize}</visualize>
+      <update_rate>${sonar.update_rate}</update_rate>
       <ray>
         <scan>
           <horizontal>
-            <samples>5</samples>
+            <samples>${sonar.h_sample}</samples>
             <resolution>1.0</resolution>
-            <min_angle>-0.25</min_angle>
-            <max_angle>0.25</max_angle>
+            <min_angle>${sonar.h_min_angle}</min_angle>
+            <max_angle>${sonar.h_max_angle}</max_angle>
           </horizontal>
           <vertical>
-            <samples>5</samples>
+            <samples>${sonar.v_sample}</samples>
             <resolution>1</resolution>
-            <min_angle>-0.25</min_angle>
-            <max_angle>0.25</max_angle>
+            <min_angle>${sonar.v_min_angle}</min_angle>
+            <max_angle>${sonar.v_max_angle}</max_angle>
           </vertical>
         </scan>
         <range>
-          <min>0.03</min>
-          <max>0.2</max>
-          <resolution>0.01</resolution>
+          <min>${sonar.min_range}</min>
+          <max>${sonar.max_range}</max>
+          <resolution>${sonar.range_res}</resolution>
         </range>
       </ray>
       <plugin name="${sonar_name}_plugin" filename="libgazebo_ros_range.so">
-        <gaussianNoise>0.005</gaussianNoise>
+        <gaussianNoise>${sonar.g_noise}</gaussianNoise>
         <alwaysOn>true</alwaysOn>
-        <updateRate>5</updateRate>
+        <updateRate>${sonar.update_rate}</updateRate>
         <topicName>${sonar_name}</topicName>
         <frameName>${sonar_name}_link</frameName>
-        <!-- field of view = (max_angle - min_angle) -->
-        <!--               = 2 max_angle -->
-        <fov>0.5</fov>
+        <fov>${sonar.fov}</fov>
         <radiation>ultrasound</radiation>
       </plugin>

File: src/robot_description/urdf/parts_cfg/base_world_cfg.xacro (robot description, xacro)
@@ -7,4 +7,4 @@
   <xacro:property name="width" value="0.4" />
   <xacro:property name="height" value="0.3" />
-  <xacro:property name="above_groud_height" value="0.05" />
+  <xacro:property name="above_groud_height" value="0.1" />
 </robot>

File: src/robot_description/urdf/tergeo.urdf.xacro (robot description, xacro)
@@ -23,8 +23,8 @@
   <xacro:caster_model caster_name="back_caster" parent_link="body_link" />
   <!-- This macro generates left sonar -->
-  <!-- <xacro:sonar_model sonar_name="left_sonar" parent_link="body_link" sonar_xyz="0 ${width/2+0.01} 0" sonar_rpy="0 0 ${PI/2}" /> -->
+  <!-- <xacro:sonar_model sonar_name="left_sonar" parent_link="body_link" /> -->
   <!-- This macro generates right sonar -->
-  <!-- <xacro:sonar_model sonar_name="right_sonar" parent_link="body_link" sonar_xyz="0 ${-width/2-0.01} 0" sonar_rpy="0 0 ${-PI/2}" /> -->
+  <!-- <xacro:sonar_model sonar_name="right_sonar" parent_link="body_link" /> -->
   <!-- This macro generates imu -->
-  <!-- <xacro:imu_model imu_name="imu" parent_link="body_link" imu_xyz="0 0 0" imu_rpy="0 0 0" /> -->
+  <xacro:imu_model imu_name="imu" parent_link="body_link" />
 </robot>
