Commit message: decompose the whole xacro file to several macros

File: src/robot_description/urdf/parts/base_world.xacro (robot description, xacro)
@@ -2,5 +2,5 @@
 <robot xmlns:xacro="TergeoRobot" name="tergeo">
   <!-- macro to generate world and robot main body -->
-  <xacro:macro name="base_world" params="world_name body_name mass length width height wheel_radius">
+  <xacro:macro name="base_world" params="world_name body_name mass length width height above_groud_height">
     <!-- base world link in rviz -->
     <link name="${world_name}"/>
@@ -8,5 +8,5 @@
       <parent link="${world_name}"/>
       <child link="${body_name}_link"/>
-      <origin xyz="0.0 0.0 ${height/2+wheel_radius-0.01}" rpy="0 0 0"/>
+      <origin xyz="0.0 0.0 ${height/2+above_groud_height-0.01}" rpy="0 0 0"/>
     </joint>
     <link name="${body_name}_link">
@@ -27,7 +27,7 @@
         <origin xyz="0 0 0" rpy="0 0 0"/>
         <mass value="${mass}"/>
-        <inertia ixx="0.00000" ixy="0.00000" ixz="0.00000"
-                iyy="0.00000" iyz="0.00000"
-                izz="0.00000" />
+        <inertia ixx="0.00001" ixy="0.00000" ixz="0.00000"
+                iyy="0.00001" iyz="0.00000"
+                izz="0.00001" />
       </inertial>
     </link>

File: src/robot_description/urdf/t_robot_args.xacro (robot description, xacro)
@@ -11,4 +11,5 @@
   <!-- Robot body is a box, below is width, height, length of the box -->
   <!-- Length by x axis, width by y axis, height by z axis -->
+  <xacro:property name="above_groud_height" value="0.2" />
   <xacro:property name="length" value="0.7"/>
   <xacro:property name="width" value="0.4"/>

File: src/robot_description/urdf/tergeo.urdf.xacro (robot description, xacro)
@@ -8,4 +8,23 @@
   <!-- Import all the macros -->
   <xacro:include filename="$(find robot_description)/urdf/parts/*.xacro"/>
-  <xacro:base_world world_name="base_world" body_name="body" mass="${mass}" length="${length}" width="${width}" height="${height}" wheel_radius="${wheel_radius}"/>
+  <!-- This macro generates a ${body_name}_link -->
+  <xacro:base_world world_name="base_world" body_name="body" mass="${mass}" length="${length}" width="${width}" height="${height}" above_groud_height="${above_groud_height}"/>
+  <!-- This macro generates the lidar model -->
+  <xacro:lidar_model lidar_name="top_lidar16" parent_link="body_link" lidar_xyz="0 0 ${lidar_above+height/2}" lidar_rpy="0 0 0" lidar_axis="0 0 1"/>
+  <!-- This macro generates left wheel -->
+  <xacro:wheel_model wheel_name="left_wheel" parent_link="body_link" wheel_xyz="0.0 ${width/2+0.02} ${-height/2}" wheel_rpy="${-PI/2} 0 0" wheel_axis="0 0 1" />
+  <!-- This macro generates right wheel -->
+  <xacro:wheel_model wheel_name="right_wheel" parent_link="body_link" wheel_xyz="0.0 ${-width/2-0.02} ${-height/2}" wheel_rpy="${-PI/2} 0 0" wheel_axis="0 0 1" />
+  <!-- This macro setups the control -->
+  <xacro:wheel_control left_wheel_name="left_wheel" right_wheel_name="right_wheel" />
+  <!-- This macro generates front caster -->
+  <xacro:caster_model caster_name="front_caster" parent_link="body_link" caster_xyz="${length/2} 0 ${-height/2-0.05}" caster_rpy="0 0 0" />
+  <!-- This macro generates back caster -->
+  <xacro:caster_model caster_name="back_caster" parent_link="body_link" caster_xyz="${-length/2} 0 ${-height/2-0.05}" caster_rpy="0 0 0" />
+  <!-- This macro generates left sonar -->
+  <xacro:sonar_model sonar_name="left_sonar" parent_link="body_link" sonar_xyz="0 ${width/2+0.01} 0" sonar_rpy="0 0 ${PI/2}" />
+  <!-- This macro generates right sonar -->
+  <xacro:sonar_model sonar_name="right_sonar" parent_link="body_link" sonar_xyz="0 ${-width/2-0.01} 0" sonar_rpy="0 0 ${-PI/2}" />
+  <!-- This macro generates imu -->
+  <xacro:imu_model imu_name="imu" parent_link="body_link" imu_xyz="0 0 0" imu_rpy="0 0 0" />
 </robot>

Commit message: modifying

File: src/robot_description/urdf/parts/base_world.xacro (robot description, xacro)
@@ -1,6 +1,8 @@
 <?xml version="1.0"?>
 <robot xmlns:xacro="TergeoRobot" name="tergeo">
+  <!-- include corresponding config file -->
+  <xacro:include filename="$(find robot_description)/urdf/parts_cfg/base_world_cfg.xacro" ns="base" />
   <!-- macro to generate world and robot main body -->
-  <xacro:macro name="base_world" params="world_name body_name mass length width height above_groud_height">
+  <xacro:macro name="base_world" params="world_name body_name">
     <!-- base world link in rviz -->
     <link name="${world_name}"/>
@@ -8,5 +10,5 @@
       <parent link="${world_name}"/>
       <child link="${body_name}_link"/>
-      <origin xyz="0.0 0.0 ${height/2+above_groud_height-0.01}" rpy="0 0 0"/>
+      <origin xyz="0.0 0.0 ${base.height/2+base.above_groud_height}" rpy="0 0 0"/>
     </joint>
     <link name="${body_name}_link">
@@ -14,5 +16,5 @@
         <origin xyz="0.0 0.0 0.0" rpy="0 0 0"/>
         <geometry>
-          <box size="${length} ${width} ${height}"/>
+          <box size="${base.length} ${base.width} ${base.height}"/>
         </geometry>
         <material name="orange"/>
@@ -21,13 +23,13 @@
         <origin xyz="0.0 0.0 0.0" rpy="0 0 0"/>
         <geometry>
-          <box size="${length} ${width} ${height}"/>
+          <box size="${base.length} ${base.width} ${base.height}"/>
         </geometry>
       </collision>
       <inertial>
         <origin xyz="0 0 0" rpy="0 0 0"/>
-        <mass value="${mass}"/>
-        <inertia ixx="0.00001" ixy="0.00000" ixz="0.00000"
-                iyy="0.00001" iyz="0.00000"
-                izz="0.00001" />
+        <mass value="${base.mass}"/>
+        <inertia ixx="0.0000" ixy="0.00000" ixz="0.00000"
+                iyy="0.0000" iyz="0.00000"
+                izz="0.0000" />
       </inertial>
     </link>

File: src/robot_description/urdf/parts/lidar_model.xacro (robot description, xacro)
@@ -1,26 +1,17 @@
 <?xml version="1.0"?>
 <robot xmlns:xacro="TergeoRobot" name="tergeo">
-  <!-- Local args -->
-  <xacro:property name="lidar_mass" value="1.0" />
-  <xacro:property name="lidar_height" value="0.02" />
-  <xacro:property name="lidar_radius" value="0.02" />
-  <xacro:property name="h_sample" value="1800" />
-  <xacro:property name="h_min_angle" value="${-180*3.1415926535897931/180.0}" />
-  <xacro:property name="h_max_angle" value="${+180*3.1415926535897931/180.0}" />
-  <xacro:property name="v_sample" value="16" />
-  <xacro:property name="v_min_angle" value="${-15.0*3.1415926535897931/180.0}" />
-  <xacro:property name="v_max_angle" value="${15.0*3.1415926535897931/180.0}" />
-  <xacro:property name="pub_topic_name" value="/sensor/lidar16/top/pointcloud" />
-  <xacro:property name="min_range" value="0.2" />
-  <xacro:property name="max_range" value="100.0" />
-  <xacro:property name="min_intensity" value="0.001" />
-  <xacro:property name="gaussian_noise" value="0.02" />
-  <!-- Macro to generate lidar -->
-  <xacro:macro name="lidar_model" params="lidar_name parent_link lidar_xyz lidar_rpy lidar_axis">
+  <!-- base cfg and lidar cfg -->
+  <xacro:include filename="$(find robot_description)/urdf/parts_cfg/lidar_cfg.xacro" ns="lidar" />
+  <xacro:include filename="$(find robot_description)/urdf/parts_cfg/base_world_cfg.xacro" ns="base" />
+  <!-- local args which need args from base cfg and lidar cfg -->
+  <!-- This arg will be deprecated soon -->
+  <xacro:property name="lidar_xyz" value="0 0 ${lidar.above_height+base.height/2+lidar.height/2}" />
+  <!-- Macro to generate lidar model -->
+  <xacro:macro name="lidar_model" params="lidar_name parent_link">
     <joint name="${lidar_name}_joint" type="fixed">
       <parent link="${parent_link}" />
       <child link="${lidar_name}_link" />
-      <origin xyz="${lidar_xyz}" rpy="${lidar_rpy}" />
-      <axis xyz="${lidar_axis}" />
+      <origin xyz="${lidar_xyz}" rpy="${lidar.rpy}" />
+      <axis xyz="${lidar.axis}" />
     </joint>
     <link name="${lidar_name}_link">
@@ -28,5 +19,5 @@
         <origin xyz="0.0 0.0 0.0" rpy="0 0 0" />
         <geometry>
-          <cylinder length="${lidar_height}" radius="${lidar_radius}" />
+          <cylinder length="${lidar.height}" radius="${lidar.radius}" />
         </geometry>
         <material name="blue" />
@@ -35,9 +26,9 @@
         <origin xyz="0.0 0.0 0.0" rpy="0 0 0" />
         <geometry>
-          <cylinder length="${lidar_height}" radius="${lidar_radius}" />
+          <cylinder length="${lidar.height}" radius="${lidar.radius}" />
         </geometry>
       </collision>
       <inertial>
-        <mass value="${lidar_mass}" />
+        <mass value="${lidar.mass}" />
         <origin xyz="0 0 0" />
         <inertia ixx="0.0" ixy="0.0" ixz="0.0"
@@ -47,30 +38,29 @@
     </link>
     <!-- Gazebo plugin for lidar -->
-    <!-- robot laser setup in gazebo -->
     <gazebo reference="${lidar_name}_link">
       <material>Gazebo/Red</material>
       <sensor type="ray" name="laser_16">
         <pose>0 0 0 0 0 0</pose>
-        <visualize>false</visualize>
-        <update_rate>10</update_rate>
+        <visualize>${lidar.visualize}</visualize>
+        <update_rate>${lidar.update_rate}</update_rate>
         <ray>
           <scan>
             <horizontal>
-              <samples>${h_sample}</samples>
+              <samples>${lidar.h_sample}</samples>
               <resolution>1</resolution>
-              <min_angle>${h_min_angle}</min_angle>
-              <max_angle>${h_max_angle}</max_angle>
+              <min_angle>${lidar.h_min_angle}</min_angle>
+              <max_angle>${lidar.h_max_angle}</max_angle>
             </horizontal>
             <vertical>
-              <samples>${v_sample}</samples>
+              <samples>${lidar.v_sample}</samples>
               <resolution>1</resolution>
-              <min_angle>${v_min_angle}</min_angle>
-              <max_angle>${v_max_angle}</max_angle>
+              <min_angle>${lidar.v_min_angle}</min_angle>
+              <max_angle>${lidar.v_max_angle}</max_angle>
             </vertical>
           </scan>
           <range>
-            <min>${min_range}</min>
-            <max>${max_range}</max>
-            <resolution>0.01</resolution>
+            <min>${lidar.min_range}</min>
+            <max>${lidar.max_range}</max>
+            <resolution>${lidar.range_res}</resolution>
           </range>
           <noise>
@@ -81,10 +71,11 @@
         </ray>
         <plugin name="gazebo_ros_laser_controller" filename="libgazebo_ros_velodyne_laser.so">
-          <topicName>${pub_topic_name}</topicName>
+          <topicName>${lidar.pub_topic_name}</topicName>
           <frameName>${lidar_name}_link</frameName>
-          <min_range>${min_range}</min_range>
-          <max_range>${max_range}</max_range>
+          <min_range>${lidar.min_range}</min_range>
+          <max_range>${lidar.max_range}</max_range>
+          <!-- TODO: Not sure need this arg or not? -->
           <!-- <min_intensity>${min_intensity}</min_intensity> -->
-          <gaussianNoise>${gaussian_noise}</gaussianNoise>
+          <gaussianNoise>${lidar.gaussian_noise}</gaussianNoise>
         </plugin>
       </sensor>

File: src/robot_description/urdf/parts/wheel_model.xacro (robot description, xacro)
@@ -1,9 +1,18 @@
 <?xml version="1.0"?>
 <robot xmlns:xacro="TergeoRobot" name="tergeo">
-  <!-- args -->
-  <xacro:property name="wheel_thickness" value=" 0.02" />
-  <xacro:property name="wheel_radius" value="0.10" />
+  <!-- include corresponding config file -->
+  <xacro:include filename="$(find robot_description)/urdf/parts_cfg/wheel_cfg.xacro" ns="wheel" />
+  <xacro:include filename="$(find robot_description)/urdf/parts_cfg/base_world_cfg.xacro" ns="base" />
   <!-- Definition of the wheel macro -->
   <xacro:macro name="wheel_model" params="wheel_name parent_link wheel_xyz wheel_rpy wheel_axis">
+    <!-- args depend on macro params and cfg file -->
+    <xacro:if value="${'left' in wheel_name}">
+      <xacro:property name="wheel_xyz" value="0 +" />
+      <xacro:property name="wheel_rpy" value="" />
+    </xacro:if>
+    <xacro:if value="${'right' in wheel_name}">
+      <xacro:property name="wheel_xyz" value="" />
+      <xacro:property name="wheel_rpy" value="" />
+    </xacro:if>
     <!-- wheel joint -->
     <joint name="${wheel_name}_joint" type="continuous">
@@ -18,5 +27,5 @@
         <origin xyz="0.0 0.0 0.0" rpy="0 0 0" />
         <geometry>
-          <cylinder length="${wheel_thickness}" radius="${wheel_radius}" />
+          <cylinder length="${wheel.thickness}" radius="${wheel.radius}" />
         </geometry>
         <material name="green" />
@@ -25,21 +34,14 @@
         <origin xyz="0.0 0.0 0.0" rpy="0 0 0" />
         <geometry>
-          <cylinder length="${wheel_thickness}" radius="${wheel_radius}" />
+          <cylinder length="${wheel.thickness}" radius="${wheel.radius}" />
         </geometry>
       </collision>
       <inertial>
         <origin xyz="0 0 0" />
-        <mass value="1" />
+        <mass value="${}" />
         <inertia ixx="0.0025" ixy="0" ixz="0"
                 iyy="0.0025" iyz="0"
                 izz="0.005" />
       </inertial>
-      <!-- <inertial>
-        <origin xyz="0 0 0" />
-        <mass value="2" />
-        <inertia ixx="${0.025/2}" ixy="0" ixz="0"
-                iyy="${0.025/2}" iyz="0"
-                izz="${0.05/2}" />
-      </inertial> -->
     </link>
     <!-- setup the motor -->
@@ -85,5 +87,5 @@
         <!-- wheel seperation need to know the body width -->
         <wheelSeparation>0.46</wheelSeparation>
-        <wheelDiameter>${2*wheel_radius}</wheelDiameter>
+        <wheelDiameter>${2*wheel.radius}</wheelDiameter>
         <wheelAcceleration>100</wheelAcceleration>
         <wheelTorque>5</wheelTorque>

File: src/robot_description/urdf/tergeo.urdf.xacro (robot description, xacro)
@@ -3,5 +3,5 @@
 <robot name="tergeo" xmlns:xacro="TergeoRobot">
   <!-- Import all designed robot model args  -->
-  <xacro:include filename="$(find robot_description)/urdf/t_robot_args.xacro"/>
+  <!-- <xacro:include filename="$(find robot_description)/urdf/t_robot_args.xacro"/> -->
   <!-- Import Rviz colors -->
   <xacro:include filename="$(find robot_description)/urdf/rviz_materials.xacro"/>
@@ -9,17 +9,17 @@
   <xacro:include filename="$(find robot_description)/urdf/parts/*.xacro"/>
   <!-- This macro generates a ${body_name}_link -->
-  <xacro:base_world world_name="base_world" body_name="body" mass="${mass}" length="${length}" width="${width}" height="${height}" above_groud_height="${above_groud_height}" />
+  <xacro:base_world world_name="base_world" body_name="body" />
   <!-- This macro generates the lidar model -->
-  <xacro:lidar_model lidar_name="top_lidar16" parent_link="body_link" lidar_xyz="0 0 ${lidar_above+height/2}" lidar_rpy="0 0 0" lidar_axis="0 0 1" />
+  <xacro:lidar_model lidar_name="top_lidar16" parent_link="body_link" />
   <!-- This macro generates left wheel -->
-  <xacro:wheel_model wheel_name="left_wheel" parent_link="body_link" wheel_xyz="0.0 ${width/2+0.02} ${-height/2}" wheel_rpy="${-PI/2} 0 0" wheel_axis="0 0 1" />
+  <!-- <xacro:wheel_model wheel_name="left_wheel" parent_link="body_link" wheel_xyz="0.0 ${width/2+0.02} ${-height/2}" wheel_rpy="${-PI/2} 0 0" wheel_axis="0 0 1" /> -->
   <!-- This macro generates right wheel -->
-  <xacro:wheel_model wheel_name="right_wheel" parent_link="body_link" wheel_xyz="0.0 ${-width/2-0.02} ${-height/2}" wheel_rpy="${-PI/2} 0 0" wheel_axis="0 0 1" />
+  <!-- <xacro:wheel_model wheel_name="right_wheel" parent_link="body_link" wheel_xyz="0.0 ${-width/2-0.02} ${-height/2}" wheel_rpy="${-PI/2} 0 0" wheel_axis="0 0 1" /> -->
   <!-- This macro setups the control -->
-  <xacro:wheel_control left_wheel_name="left_wheel" right_wheel_name="right_wheel" />
+  <!-- <xacro:wheel_control left_wheel_name="left_wheel" right_wheel_name="right_wheel" /> -->
   <!-- This macro generates front caster -->
-  <xacro:caster_model caster_name="front_caster" parent_link="body_link" caster_xyz="${length/2} 0 ${-height/2-0.05}" caster_rpy="0 0 0" />
+  <!-- <xacro:caster_model caster_name="front_caster" parent_link="body_link" caster_xyz="${length/2} 0 ${-height/2-0.05}" caster_rpy="0 0 0" /> -->
   <!-- This macro generates back caster -->
-  <xacro:caster_model caster_name="back_caster" parent_link="body_link" caster_xyz="${-length/2} 0 ${-height/2-0.05}" caster_rpy="0 0 0" />
+  <!-- <xacro:caster_model caster_name="back_caster" parent_link="body_link" caster_xyz="${-length/2} 0 ${-height/2-0.05}" caster_rpy="0 0 0" /> -->
   <!-- This macro generates left sonar -->
   <!-- <xacro:sonar_model sonar_name="left_sonar" parent_link="body_link" sonar_xyz="0 ${width/2+0.01} 0" sonar_rpy="0 0 ${PI/2}" /> -->
@@ -27,4 +27,4 @@
   <!-- <xacro:sonar_model sonar_name="right_sonar" parent_link="body_link" sonar_xyz="0 ${-width/2-0.01} 0" sonar_rpy="0 0 ${-PI/2}" /> -->
   <!-- This macro generates imu -->
-  <xacro:imu_model imu_name="imu" parent_link="body_link" imu_xyz="0 0 0" imu_rpy="0 0 0" />
+  <!-- <xacro:imu_model imu_name="imu" parent_link="body_link" imu_xyz="0 0 0" imu_rpy="0 0 0" /> -->
 </robot>
