Commit message: update xmlns, add turtlebot and robot_control

File: src/robot_description/urdf/parts/base_world.xacro (robot description, xacro)
@@ -1,4 +1,4 @@
 <?xml version="1.0"?>
-<robot xmlns:xacro="TergeoRobot" name="tergeo">
+<robot xmlns:xacro="http://ros.org/wiki/xacro" name="tergeo">
   <!-- include corresponding config file -->
   <xacro:include filename="$(find robot_description)/urdf/parts_cfg/base_world_cfg.xacro" ns="base" />

File: src/robot_description/urdf/parts/caster_model.xacro (robot description, xacro)
@@ -1,4 +1,4 @@
 <?xml version="1.0"?>
-<robot xmlns:xacro="TergeoRobot" name="tergeo">
+<robot xmlns:xacro="http://ros.org/wiki/xacro" name="tergeo">
   <!-- Import args -->
   <xacro:include filename="$(find robot_description)/urdf/parts_cfg/base_world_cfg.xacro" ns="base" />
@@ -49,4 +49,5 @@
       <maxVel>${caster.max_vel}</maxVel>
       <material>Gazebo/FlatBlack</material>
+      <selfCollide>false</selfCollide>
     </gazebo>
   </xacro:macro>

File: src/robot_description/urdf/parts/imu_model.xacro (robot description, xacro)
@@ -1,4 +1,4 @@
 <?xml version="1.0"?>
-<robot xmlns:xacro="TergeoRobot" name="tergeo">
+<robot xmlns:xacro="http://ros.org/wiki/xacro" name="tergeo">
   <!-- args -->
   <xacro:include filename="$(find robot_description)/urdf/parts_cfg/imu_cfg.xacro" ns="imu" />

File: src/robot_description/urdf/parts/lidar_model.xacro (robot description, xacro)
@@ -1,4 +1,4 @@
 <?xml version="1.0"?>
-<robot xmlns:xacro="TergeoRobot" name="tergeo">
+<robot xmlns:xacro="http://ros.org/wiki/xacro" name="tergeo">
   <!-- base cfg and lidar cfg -->
   <xacro:include filename="$(find robot_description)/urdf/parts_cfg/lidar_cfg.xacro" ns="lidar" />

File: src/robot_description/urdf/parts/sonar_model.xacro (robot description, xacro)
@@ -1,4 +1,4 @@
 <?xml version="1.0"?>
-<robot xmlns:xacro="TergeoRobot" name="tergeo">
+<robot xmlns:xacro="http://ros.org/wiki/xacro" name="tergeo">
 <xacro:include filename="$(find robot_description)/urdf/parts_cfg/sonar_cfg.xacro" ns="sonar" />
 <xacro:macro name="sonar_model" params="sonar_name parent_link">

File: src/robot_description/urdf/parts/wheel_model.xacro (robot description, xacro)
@@ -1,4 +1,4 @@
 <?xml version="1.0"?>
-<robot xmlns:xacro="TergeoRobot" name="tergeo">
+<robot xmlns:xacro="http://ros.org/wiki/xacro" name="tergeo">
   <!-- include corresponding config file -->
   <xacro:include filename="$(find robot_description)/urdf/parts_cfg/base_world_cfg.xacro" ns="base" />
@@ -47,9 +47,9 @@
       <type>transmission_interface/SimpleTransmission</type>
       <joint name="${wheel_name}_joint">
-        <hardwareInterface>VelocityJointInterface</hardwareInterface>
+        <hardwareInterface>hardware_interface/EffortJointInterface</hardwareInterface>
       </joint>
       <actuator name="${wheel_name}_motor">
-        <hardwareInterface>VelocityJointInterface</hardwareInterface>
-        <mechanicalReduction>1</mechanicalReduction>
+        <hardwareInterface>hardware_interface/EffortJointInterface</hardwareInterface>
+        <mechanicalReduction>0.5</mechanicalReduction>
       </actuator>
     </transmission>
@@ -90,4 +90,9 @@
       </plugin>
     </gazebo>
+    <gazebo>
+      <plugin name="gazebo_ros_control" filename="libgazebo_ros_control.so">
+        <robotNamespace>/rjptest</robotNamespace>
+      </plugin>
+    </gazebo>
   </xacro:macro>
 </robot>

File: src/robot_description/urdf/parts_cfg/base_world_cfg.xacro (robot description, xacro)
@@ -2,5 +2,5 @@
 <!-- Tergeo Washing Floor Robot -->
 <!-- args for base_world model -->
-<robot name="tergeo" xmlns:xacro="TergeoRobot">
+<robot name="tergeo" xmlns:xacro="http://ros.org/wiki/xacro">
   <xacro:property name="mass" value="200" />
   <xacro:property name="length" value="0.7" />

File: src/robot_description/urdf/parts_cfg/caster_cfg.xacro (robot description, xacro)
@@ -1,4 +1,4 @@
 <?xml version="1.0" ?>
-<robot name="tergeo" xmlns:xacro="TergeoRobot">
+<robot name="tergeo" xmlns:xacro="http://ros.org/wiki/xacro">
   <!-- Arg depends on cfg file -->
   <xacro:include filename="$(find robot_description)/urdf/parts_cfg/wheel_cfg.xacro" ns="wheel" />
@@ -7,8 +7,8 @@
   <xacro:property name="width" value="0.03" />
   <xacro:property name="rpy" value="0 0 0" />
-  <!-- Wheel intrinsic -->
-  <xacro:property name="mass" value="1.0" />
-  <xacro:property name="mu1" value="0.1" />
-  <xacro:property name="mu2" value="0.1" />
+  <!-- Caster intrinsic -->
+  <xacro:property name="mass" value="0.1" />
+  <xacro:property name="mu1" value="0.0" />
+  <xacro:property name="mu2" value="0.0" />
   <xacro:property name="kp" value="500000.0" />
   <xacro:property name="kd" value="10.0" />

File: src/robot_description/urdf/parts_cfg/imu_cfg.xacro (robot description, xacro)
@@ -1,4 +1,4 @@
 <?xml version="1.0" ?>
-<robot name="tergeo" xmlns:xacro="TergeoRobot">
+<robot name="tergeo" xmlns:xacro="http://ros.org/wiki/xacro">
   <xacro:property name="always_on" value="true" />
   <xacro:property name="topic_name" value="imu" />

File: src/robot_description/urdf/parts_cfg/lidar_cfg.xacro (robot description, xacro)
@@ -1,4 +1,4 @@
 <?xml version="1.0"?>
-<robot name="tergeo" xmlns:xacro="TergeoRobot">
+<robot name="tergeo" xmlns:xacro="http://ros.org/wiki/xacro">
   <!-- Import the cfg -->
   <xacro:include filename="$(find robot_description)/urdf/parts_cfg/base_world_cfg.xacro" ns="base" />

File: src/robot_description/urdf/parts_cfg/sonar_cfg.xacro (robot description, xacro)
@@ -1,4 +1,4 @@
 <?xml version="1.0" ?>
-<robot name="tergeo" xmlns:xacro="TergeoRobot">
+<robot name="tergeo" xmlns:xacro="http://ros.org/wiki/xacro">
   <xacro:include filename="$(find robot_description)/urdf/parts_cfg/base_world_cfg.xacro" ns="base" />
   <!-- Math -->

File: src/robot_description/urdf/parts_cfg/wheel_cfg.xacro (robot description, xacro)
@@ -1,8 +1,8 @@
 <?xml version="1.0"?>
-<robot name="tergeo" xmlns:xacro="TergeoRobot">
+<robot name="tergeo" xmlns:xacro="http://ros.org/wiki/xacro">
   <!-- Math args -->
   <xacro:property name="PI" value="3.1415926535897931" />
   <!-- Wheel extrinsic -->
-  <xacro:property name="rpy" value="${-PI/2} 0 0" />
+  <xacro:property name="rpy" value="${-PI/2} 0 0" />`
   <xacro:property name="axis" value="0 0 1" />
   <xacro:property name="mass" value="1.00" />
@@ -16,6 +16,6 @@
   <xacro:property name="z_dis" value="0.05" />
   <!-- Wheel intrinsic -->
-  <xacro:property name="mu1" value="0.1" />
-  <xacro:property name="mu2" value="0.1" />
+  <xacro:property name="mu1" value="50.0" />
+  <xacro:property name="mu2" value="50.0" />
   <xacro:property name="kp" value="500000.0" />
   <xacro:property name="kd" value="10.0" />
@@ -29,5 +29,5 @@
   <xacro:property name="odom_src" value="world" />
   <xacro:property name="update_rate" value="30" />
-  <xacro:property name="accel" value="1000" />
+  <xacro:property name="accel" value="1" />
   <xacro:property name="torque" value="5" />
 </robot>

File: src/robot_description/urdf/tergeo.urdf.xacro (robot description, xacro)
@@ -1,5 +1,5 @@
 <?xml version="1.0"?>
 <!-- Tergeo Washing Floor Robot -->
-<robot name="tergeo" xmlns:xacro="TergeoRobot">
+<robot name="tergeo" xmlns:xacro="http://ros.org/wiki/xacro">
   <!-- Import all designed robot model args  -->
   <!-- <xacro:include filename="$(find robot_description)/urdf/t_robot_args.xacro"/> -->
