Commit message: add tb_modify_dsecription

File: src/tb_modify_description/urdf/my_burger.gazebo.xacro (robot description, xacro)
@@ -4,5 +4,5 @@
   <xacro:arg name="imu_visual"   default="false"/>
   <gazebo reference="base_link">
-    <material>Gazebo/DarkGrey</material>
+    <material>Gazebo/Orange</material>
   </gazebo>
   <gazebo reference="wheel_left_link">
@@ -14,5 +14,5 @@
     <maxVel>0.1</maxVel>
     <fdir1>1 0 0</fdir1>
-    <material>Gazebo/FlatBlack</material>
+    <material>Gazebo/DarkYellow</material>
   </gazebo>
   <gazebo reference="wheel_right_link">
@@ -24,5 +24,5 @@
     <maxVel>0.1</maxVel>
     <fdir1>1 0 0</fdir1>
-    <material>Gazebo/FlatBlack</material>
+    <material>Gazebo/DarkYellow</material>
   </gazebo>
   <gazebo reference="caster_back_link">
@@ -125,6 +125,6 @@
         </ray>
         <plugin name="gazebo_ros_laser_controller" filename="libgazebo_ros_velodyne_laser.so">
-          <topicName>mypt2</topicName>
-          <frameName>base_scan_link</frameName>
+          <topicName>/mypt2</topicName>
+          <frameName>base_scan</frameName>
           <min_range>0.2</min_range>
           <max_range>5</max_range>

File: src/tb_modify_description/urdf/my_burger.urdf.xacro (robot description, xacro)
@@ -2,5 +2,5 @@
 <robot name="turtlebot3_burger" xmlns:xacro="http://ros.org/wiki/xacro">
   <xacro:include filename="$(find tb_modify_description)/urdf/common_properties.xacro"/>
-  <xacro:include filename="$(find tb_modify_description)/urdf/turtlebot3_burger.gazebo.xacro"/>
+  <xacro:include filename="$(find tb_modify_description)/urdf/my_burger.gazebo.xacro"/>
   <link name="base_footprint"/>
   <joint name="base_joint" type="fixed">
@@ -11,7 +11,8 @@
   <link name="base_link">
     <visual>
-      <origin xyz="-0.032 0 0.0" rpy="0 0 0"/>
+      <origin xyz="-0.032 0 0.20" rpy="0 0 0"/>
       <geometry>
-        <mesh filename="package://tb_modify_description/meshes/bases/burger_base.stl" scale="0.001 0.001 0.001"/>
+        <box size="0.7 0.4 0.3"/>
+        <!-- <mesh filename="package://tb_modify_description/meshes/bases/burger_base.stl" scale="0.001 0.001 0.001"/> -->
       </geometry>
       <material name="light_black"/>

Commit message: add script and fix turtlebot

File: src/tb_modify_description/urdf/my_burger.gazebo.xacro (robot description, xacro)
@@ -124,5 +124,5 @@
           </noise>
         </ray>
-        <plugin name="gazebo_ros_laser_controller" filename="libgazebo_ros_velodyne_laser.so">
+        <plugin name="lidar_sensor" filename="libgazebo_ros_velodyne_laser.so">
           <topicName>/mypt2</topicName>
           <frameName>base_scan</frameName>

File: src/tb_modify_description/urdf/my_burger.urdf.xacro (robot description, xacro)
@@ -18,4 +18,5 @@
       <material name="light_black"/>
     </visual>
+    <!-- old collision-->
     <collision>
       <origin xyz="-0.032 0 0.070" rpy="0 0 0"/>
@@ -24,4 +25,12 @@
       </geometry>
     </collision>
+    <!-- test collision -->
+    <!-- <collision>
+      <origin xyz="-0.032 0 0.20" rpy="0 0 0"/>
+      <geometry>
+        <box size="0.7 0.4 0.3"/>
+      </geometry>
+      <material name="light_black"/>
+    </collision> -->
     <inertial>
       <origin xyz="0 0 0" rpy="0 0 0"/>
@@ -117,5 +126,6 @@
     <parent link="base_link"/>
     <child link="base_scan"/>
-    <origin xyz="-0.032 0 0.172" rpy="0 0 0"/>
+    <!-- <origin xyz="-0.032 0 0.172" rpy="0 0 0"/> -->
+    <origin xyz="-0.032 0 0.472" rpy="0 0 0"/>
   </joint>
   <link name="base_scan">
