Commit message: update, modify turtlebot3

File: src/tb_modify_description/urdf/my_burger.urdf.xacro (robot description, xacro)
@@ -67,5 +67,5 @@
                iyy="1.1192413e-05" iyz="-1.4400107e-11"
                izz="2.0712558e-05" />
-      </inertial>
+    </inertial>
   </link>
   <joint name="wheel_right_joint" type="continuous">
