Commit message: finished tergeo_teleop package but still have control problems

File: src/tergeo_description/urdf/macro/cfg/cfg_lidar.xacro (robot description, xacro)
@@ -18,5 +18,5 @@
   <xacro:property name="gaussian_noise" value="0.02" />
   <!-- others -->
-  <xacro:property name="visualize" value="true" />
+  <xacro:property name="visualize" value="false" />
   <xacro:property name="update_rate" value="10" />
   <xacro:property name="pub_topic_name" value="/sensor/lidar16/top/pointcloud" />

File: src/tergeo_description/urdf/tergeo.urdf.xacro (robot description, xacro)
@@ -12,6 +12,6 @@
   <xacro:control_model left_wheel_name="left_wheel" right_wheel_name="right_wheel" world_link="base_world" />
   <xacro:caster_model caster_name="back_caster" parent_link="base_link" />
-  <xacro:imu_model imu_name="imu" parent_link="base_link" />
-  <xacro:sonar_model sonar_name="left_sonar" parent_link="base_link" />
-  <xacro:sonar_model sonar_name="right_sonar" parent_link="base_link" />
+  <!-- <xacro:imu_model imu_name="imu" parent_link="base_link" /> -->
+  <!-- <xacro:sonar_model sonar_name="left_sonar" parent_link="base_link" /> -->
+  <!-- <xacro:sonar_model sonar_name="right_sonar" parent_link="base_link" /> -->
 </robot>
