Commit message: finished tergeo_description package

File: src/tergeo_description/urdf/macro/cfg/cfg_sonar.xacro (robot description, xacro)
@@ -1,5 +1,5 @@
 <?xml version="1.0" ?>
 <robot name="tergeo" xmlns:xacro="http://ros.org/wiki/xacro">
-  <xacro:include filename="$(find tb_modify_description)/urdf/macro/cfg_base.xacro" ns="base" />
+  <xacro:include filename="$(find tergeo_description)/urdf/macro/cfg/cfg_base.xacro" ns="base" />
   <!-- Math -->
   <xacro:property name="PI" value="3.1415926535897931" />
@@ -7,7 +7,7 @@
   <!-- Append the sonars you need -->
   <!-- Here is only 2 examples for simple car -->
-  <xacro:property name="left_xyz" value="0 ${+(base.width/2+0.01)} 0" />
+  <xacro:property name="left_xyz" value="0 ${+(base.width/2+0.01)} ${0.033+base.height/2}" />
   <xacro:property name="left_rpy" value="0 0 ${PI/2}" />
-  <xacro:property name="right_xyz" value="0 ${-(base.width/2+0.01)} 0" />
+  <xacro:property name="right_xyz" value="0 ${-(base.width/2+0.01)} ${0.033+base.height/2}" />
   <xacro:property name="right_rpy" value="0 0 ${-PI/2}" />
   <!-- sonar size is fixed to -->

File: src/tergeo_description/urdf/macro/model_base.xacro (robot description, xacro)
@@ -4,13 +4,13 @@
   <xacro:include filename="$(find tergeo_description)/urdf/macro/cfg/cfg_base.xacro" ns="base" />
   <!-- Macro to generate base model -->
-  <!-- Input base_name and parent_link -->
+  <!-- Input base_name and world_link -->
   <!-- EXAMPLE
-    <xacro:basemodel base_name="base" parent_link="world" />
+    <xacro:basemodel base_name="base" world_link="world" />
     It will generate a `base_link` and `world`
   -->
-  <xacro:macro name="base_model" params="base_name parent_link">
-    <link name="${parent_link}"/>
+  <xacro:macro name="base_model" params="base_name world_link">
+    <link name="${world_link}"/>
     <joint name="${base_name}_joint" type="fixed">
-      <parent link="${parent_link}"/>
+      <parent link="${world_link}"/>
       <child link="${base_name}_link"/>
       <origin xyz="0.0 0.0 0.010" rpy="0 0 0"/>

File: src/tergeo_description/urdf/macro/model_sonar.xacro (robot description, xacro)
@@ -1,13 +1,13 @@
 <?xml version="1.0"?>
 <robot name="tergeo" xmlns:xacro="http://ros.org/wiki/xacro">
-<xacro:include filename="$(find tb_modify_description)/urdf/macro/cfg_sonar.xacro" ns="sonar" />
+<xacro:include filename="$(find tergeo_description)/urdf/macro/cfg/cfg_sonar.xacro" ns="sonar" />
 <xacro:macro name="sonar_model" params="sonar_name parent_link">
   <xacro:if value="${'left' in sonar_name}">
-      <xacro:property name="sonar_xyz" value="${sonar.left_xyz}" />
-      <xacro:property name="sonar_rpy" value="${sonar.left_rpy}" />
+    <xacro:property name="sonar_xyz" value="${sonar.left_xyz}" />
+    <xacro:property name="sonar_rpy" value="${sonar.left_rpy}" />
   </xacro:if>
   <xacro:if value="${'right' in sonar_name}">
-      <xacro:property name="sonar_xyz" value="${sonar.right_xyz}" />
-      <xacro:property name="sonar_rpy" value="${sonar.right_rpy}" />
+    <xacro:property name="sonar_xyz" value="${sonar.right_xyz}" />
+    <xacro:property name="sonar_rpy" value="${sonar.right_rpy}" />
   </xacro:if>
   <!-- sonar joint -->
@@ -34,5 +34,5 @@
     <inertial>
       <origin xyz="0 0 0" />
-      <mass value="0.001" />
+      <mass value="0.000001" />
       <inertia ixx="0.000" ixy="0.0" ixz="0.0"
                iyy="0.000" iyz="0.0"

File: src/tergeo_description/urdf/macro/model_wheel.xacro (robot description, xacro)
@@ -2,5 +2,83 @@
 <robot name="tergeo" xmlns:xacro="http://ros.org/wiki/xacro">
   <!-- Import  -->
-  <xacro:include filename="$(find tergeo_description)/urdf/macro/cfg/cfg_lidar.xacro" ns="lidar" />
-  <!-- Macro to generate lidar -->
+  <xacro:include filename="$(find tergeo_description)/urdf/macro/cfg/cfg_control.xacro" ns="control" />
+  <!-- Macro to generate wheel -->
+  <xacro:macro name="wheel_model" params="wheel_name parent_link">
+    <xacro:if value="${'left' in wheel_name}">
+      <xacro:property name="wheel_xyz" value="0 0.08 0.023" />
+    </xacro:if>
+    <xacro:if value="${'right' in wheel_name}">
+      <xacro:property name="wheel_xyz" value="0 -0.08 0.023" />
+    </xacro:if>
+    <joint name="${wheel_name}_joint" type="continuous">
+      <parent link="${parent_link}"/>
+      <child link="${wheel_name}_link"/>
+      <origin xyz="${wheel_xyz}" rpy="-1.57 0 0"/>
+      <axis xyz="0 0 1"/>
+    </joint>
+    <link name="${wheel_name}_link">
+      <visual>
+        <origin xyz="0 0 0" rpy="1.57 0 0"/>
+        <geometry>
+          <mesh filename="package://tergeo_description/meshes/wheels/left_tire.stl" scale="0.001 0.001 0.001"/>
+        </geometry>
+        <material name="dark"/>
+      </visual>
+      <collision>
+        <origin xyz="0 0 0" rpy="0 0 0"/>
+        <geometry>
+          <cylinder length="0.018" radius="0.033"/>
+        </geometry>
+      </collision>
+      <inertial>
+        <origin xyz="0 0 0" />
+        <mass value="2.8498940e-02" />
+        <inertia ixx="1.1175580e-05" ixy="-4.2369783e-11" ixz="-5.9381719e-09"
+                iyy="1.1192413e-05" iyz="-1.4400107e-11"
+                izz="2.0712558e-05" />
+      </inertial>
+    </link>
+    <!-- gazebo element -->
+    <gazebo reference="${wheel_name}_link">
+      <mu1>0.1</mu1>
+      <mu2>0.1</mu2>
+      <kp>500000.0</kp>
+      <kd>10.0</kd>
+      <minDepth>0.001</minDepth>
+      <maxVel>0.1</maxVel>
+      <fdir1>1 0 0</fdir1>
+      <material>Gazebo/Green</material>
+    </gazebo>
+  </xacro:macro>
+  <!-- Macro to control the motion of the robot -->
+  <!--
+    01. `left_wheel_name` and `right_wheel_name`
+    should be same with the param `wheel_name` of the macro `wheel_model`
+    02 .`world_link`
+    should be same with the param `world_link` of the macro `base_model`
+  -->
+  <xacro:macro name="control_model" params="left_wheel_name right_wheel_name world_link">
+    <gazebo>
+      <plugin name="tergeo_controller" filename="libgazebo_ros_diff_drive.so">
+        <commandTopic>${control.sub_cmd_topic}</commandTopic>
+        <odometryTopic>${control.pub_odom_topic}</odometryTopic>
+        <odometryFrame>${control.odom_frame}</odometryFrame>
+        <odometrySource>${control.odom_source}</odometrySource>
+        <publishOdomTF>true</publishOdomTF>
+        <robotBaseFrame>${world_link}</robotBaseFrame>
+        <publishWheelTF>false</publishWheelTF>
+        <publishTf>true</publishTf>
+        <publishWheelJointState>true</publishWheelJointState>
+        <legacyMode>false</legacyMode>
+        <updateRate>${control.update_rate}</updateRate>
+        <leftJoint>${left_wheel_name}_joint</leftJoint>
+        <rightJoint>${right_wheel_name}_joint</rightJoint>
+        <wheelSeparation>0.160</wheelSeparation>
+        <wheelDiameter>0.066</wheelDiameter>
+        <wheelAcceleration>${control.accel}</wheelAcceleration>
+        <wheelTorque>${control.torque}</wheelTorque>
+        <rosDebugLevel>na</rosDebugLevel>
+      </plugin>
+    </gazebo>
+  </xacro:macro>
 </robot>

File: src/tergeo_description/urdf/test.xacro (robot description, xacro)
@@ -5,5 +5,13 @@
   <!-- Import macro -->
   <xacro:include filename="$(find tergeo_description)/urdf/macro/*.xacro" />
-  <xacro:base_model base_name="base" parent_link="world" />
+  <!-- Use macros to generate the whole robot -->
+  <xacro:base_model base_name="base" world_link="base_world" />
   <xacro:lidar_model lidar_name="lidar" parent_link="base_link" />
+  <xacro:wheel_model wheel_name="left_wheel" parent_link="base_link" />
+  <xacro:wheel_model wheel_name="right_wheel" parent_link="base_link" />
+  <xacro:control_model left_wheel_name="left_wheel" right_wheel_name="right_wheel" world_link="base_world" />
+  <xacro:caster_model caster_name="back_caster" parent_link="base_link" />
+  <xacro:imu_model imu_name="imu" parent_link="base_link" />
+  <xacro:sonar_model sonar_name="left_sonar" parent_link="base_link" />
+  <xacro:sonar_model sonar_name="right_sonar" parent_link="base_link" />
 </robot>

Commit message: update

File: src/tergeo_description/urdf/macro/cfg/cfg_sonar.xacro (robot description, xacro)
@@ -14,5 +14,5 @@
   <!-- length:0.01, width:0.01, height:0.01 -->
   <!-- sonar mass is fixed to 0.01 kg -->
-  <xacro:property name="visualize" value="true" />
+  <xacro:property name="visualize" value="false" />
   <xacro:property name="update_rate" value="5" />
   <!-- fov unit is degree, positive value-->

File: src/tergeo_description/urdf/tergeo.urdf.xacro (robot description, xacro)
@@ -13,5 +13,5 @@
   <xacro:caster_model caster_name="back_caster" parent_link="base_link" />
   <xacro:imu_model imu_name="imu" parent_link="base_link" />
-  <xacro:sonar_model sonar_name="left_sonar" parent_link="base_link" />
-  <xacro:sonar_model sonar_name="right_sonar" parent_link="base_link" />
+  <!-- <xacro:sonar_model sonar_name="left_sonar" parent_link="base_link" /> -->
+  <!-- <xacro:sonar_model sonar_name="right_sonar" parent_link="base_link" /> -->
 </robot>
