Commit message: update the macro

File: src/tergeo_description/urdf/macro/cfg/cfg_base.xacro (robot description, xacro)
@@ -4,6 +4,6 @@
 <robot name="tergeo" xmlns:xacro="http://ros.org/wiki/xacro">
   <!-- visual size of the robot  -->
-  <xacro:property name="length" value="0.7" />
-  <xacro:property name="width" value="0.4" />
+  <xacro:property name="length" value="1.0" />
+  <xacro:property name="width" value="0.6" />
   <xacro:property name="height" value="0.3" />
 </robot>

File: src/tergeo_description/urdf/macro/cfg/cfg_lidar.xacro (robot description, xacro)
@@ -2,5 +2,5 @@
 <robot name="tergeo" xmlns:xacro="http://ros.org/wiki/xacro">
   <!-- Position -->
-  <xacro:property name="height" value="0.3" />
+  <xacro:property name="height" value="0.5" />
   <!-- Math args -->
   <xacro:property name="PI" value="3.1415926535897931" />
@@ -13,10 +13,10 @@
   <xacro:property name="v_max_angle" value="${+15.0 *PI/180.0}" />
   <xacro:property name="min_range" value="0.2" />
-  <xacro:property name="max_range" value="100.0" />
+  <xacro:property name="max_range" value="50.0" />
   <xacro:property name="range_res" value="0.01" />
   <xacro:property name="min_intensity" value="0.001" />
   <xacro:property name="gaussian_noise" value="0.02" />
   <!-- others -->
-  <xacro:property name="visualize" value="false" />
+  <xacro:property name="visualize" value="true" />
   <xacro:property name="update_rate" value="10" />
   <xacro:property name="pub_topic_name" value="/sensor/lidar16/top/pointcloud" />
