Commit message: update, setup PI

File: src/tergeo_description/urdf/macro/model_caster.xacro (robot description, xacro)
@@ -2,14 +2,10 @@
 <robot name="tergeo" xmlns:xacro="http://ros.org/wiki/xacro">
   <!-- Macro to generate caster model -->
-  <!-- Input base_name and world_link -->
-  <!-- EXAMPLE
-    <xacro:basemodel base_name="base" world_link="world" />
-    It will generate a `base_link` and `world`
-  -->
+  <xacro:property name="PI" value="3.1415926535897931" />
   <xacro:macro name="caster_model" params="caster_name parent_link">
     <joint name="${caster_name}_joint" type="fixed">
       <parent link="${parent_link}"/>
       <child link="${caster_name}_link"/>
-      <origin xyz="-0.081 0 -0.004" rpy="-1.57 0 0"/>
+      <origin xyz="-0.081 0 -0.004" rpy="${-PI/2} 0 0"/>
     </joint>
     <link name="${caster_name}_link">

File: src/tergeo_description/urdf/macro/model_imu.xacro (robot description, xacro)
@@ -3,10 +3,5 @@
   <!-- Import imu params -->
   <xacro:include filename="$(find tergeo_description)/urdf/macro/cfg/cfg_imu.xacro" ns="imu" />
-  <!-- Macro to generate caster model -->
-  <!-- Input base_name and world_link -->
-  <!-- EXAMPLE
-    <xacro:basemodel base_name="base" world_link="world" />
-    It will generate a `base_link` and `world`
-  -->
+  <!-- Macro to generate imu model -->
   <xacro:macro name="imu_model" params="imu_name parent_link">
     <joint name="${imu_name}_joint" type="fixed">

File: src/tergeo_description/urdf/macro/model_lidar.xacro (robot description, xacro)
@@ -9,9 +9,9 @@
       <child link="${lidar_name}_link"/>
       <!-- <origin xyz="-0.032 0 0.172" rpy="0 0 0"/> -->
-      <origin xyz="-0.032 0 ${0.172+lidar.height}" rpy="0 0 0"/>
+      <origin xyz="-0.032 0 0.172" rpy="0 0 0"/>
     </joint>
     <link name="${lidar_name}_link">
       <visual>
-        <origin xyz="0 0 0.0" rpy="0 0 0"/>
+        <origin xyz="0 0 ${lidar.height}" rpy="0 0 0"/>
         <geometry>
           <mesh filename="package://tergeo_description/meshes/sensors/lds.stl" scale="0.001 0.001 0.001"/>
@@ -26,9 +26,9 @@
       </collision>
       <inertial>
-        <mass value="0.114" />
+        <mass value="0.0114" />
         <origin xyz="0 0 0" />
-        <inertia ixx="0.001" ixy="0.0" ixz="0.0"
-                iyy="0.001" iyz="0.0"
-                izz="0.001" />
+        <inertia ixx="0.0001" ixy="0.0" ixz="0.0"
+                iyy="0.0001" iyz="0.0"
+                izz="0.0001" />
       </inertial>
     </link>

File: src/tergeo_description/urdf/macro/model_sonar.xacro (robot description, xacro)
@@ -2,4 +2,5 @@
 <robot name="tergeo" xmlns:xacro="http://ros.org/wiki/xacro">
 <xacro:include filename="$(find tergeo_description)/urdf/macro/cfg/cfg_sonar.xacro" ns="sonar" />
+<!-- Macro to generate lidar -->
 <xacro:macro name="sonar_model" params="sonar_name parent_link">
   <xacro:if value="${'left' in sonar_name}">

File: src/tergeo_description/urdf/macro/model_wheel.xacro (robot description, xacro)
@@ -4,4 +4,5 @@
   <xacro:include filename="$(find tergeo_description)/urdf/macro/cfg/cfg_control.xacro" ns="control" />
   <!-- Macro to generate wheel -->
+  <xacro:property name="PI" value="3.1415926535897931" />
   <xacro:macro name="wheel_model" params="wheel_name parent_link">
     <xacro:if value="${'left' in wheel_name}">
@@ -14,10 +15,10 @@
       <parent link="${parent_link}"/>
       <child link="${wheel_name}_link"/>
-      <origin xyz="${wheel_xyz}" rpy="-1.57 0 0"/>
+      <origin xyz="${wheel_xyz}" rpy="${-PI/2} 0 0"/>
       <axis xyz="0 0 1"/>
     </joint>
     <link name="${wheel_name}_link">
       <visual>
-        <origin xyz="0 0 0" rpy="1.57 0 0"/>
+        <origin xyz="0 0 0" rpy="${PI/2} 0 0"/>
         <geometry>
           <mesh filename="package://tergeo_description/meshes/wheels/left_tire.stl" scale="0.001 0.001 0.001"/>

File: src/tergeo_description/urdf/tergeo.urdf.xacro (robot description, xacro)
@@ -12,5 +12,5 @@
   <xacro:control_model left_wheel_name="left_wheel" right_wheel_name="right_wheel" world_link="base_world" />
   <xacro:caster_model caster_name="back_caster" parent_link="base_link" />
-  <!-- <xacro:imu_model imu_name="imu" parent_link="base_link" /> -->
+  <xacro:imu_model imu_name="imu" parent_link="base_link" />
   <!-- <xacro:sonar_model sonar_name="left_sonar" parent_link="base_link" /> -->
   <!-- <xacro:sonar_model sonar_name="right_sonar" parent_link="base_link" /> -->
