Commit message: fix control problem by setting PI to 3.1415926

File: src/tergeo_description/urdf/macro/model_lidar.xacro (robot description, xacro)
@@ -9,9 +9,9 @@
       <child link="${lidar_name}_link"/>
       <!-- <origin xyz="-0.032 0 0.172" rpy="0 0 0"/> -->
-      <origin xyz="-0.032 0 0.172" rpy="0 0 0"/>
+      <origin xyz="-0.032 0 ${lidar.height+0.172}" rpy="0 0 0"/>
     </joint>
     <link name="${lidar_name}_link">
       <visual>
-        <origin xyz="0 0 ${lidar.height}" rpy="0 0 0"/>
+        <origin xyz="0 0 0" rpy="0 0 0"/>
         <geometry>
           <mesh filename="package://tergeo_description/meshes/sensors/lds.stl" scale="0.001 0.001 0.001"/>

File: src/tergeo_description/urdf/tergeo.urdf.xacro (robot description, xacro)
@@ -13,5 +13,5 @@
   <xacro:caster_model caster_name="back_caster" parent_link="base_link" />
   <xacro:imu_model imu_name="imu" parent_link="base_link" />
-  <!-- <xacro:sonar_model sonar_name="left_sonar" parent_link="base_link" /> -->
-  <!-- <xacro:sonar_model sonar_name="right_sonar" parent_link="base_link" /> -->
+  <xacro:sonar_model sonar_name="left_sonar" parent_link="base_link" />
+  <xacro:sonar_model sonar_name="right_sonar" parent_link="base_link" />
 </robot>
